Commit message: finished part F

File: body.urdf (robot description, URDF)
Before this commit: robot robot, 3 links, 2 joints
Links:
- removed link Link0
- removed link Link1
- removed link Link2
- added link BackLeg, mass 1; collision box size=1 1 1; visual box size=1 1 1
- added link FrontLeg, mass 1; collision box size=1 1 1; visual box size=1 1 1
- added link Torso, mass 1; collision box size=1 1 1; visual box size=1 1 1
Joints:
- removed joint Link0_Link1
- removed joint Link1_Link2
- added joint Torso_BackLeg: type revolute, parent Torso, child BackLeg, origin xyz=-0.5 0 0.5 rpy=0 0 0, axis 0 1 0, limit lower=-3.14159 upper=3.14159 effort=0.0 velocity=0.0
- added joint Torso_FrontLeg: type revolute, parent Torso, child FrontLeg, origin xyz=0.5 0 0.5 rpy=0 0 0, axis 0 1 0, limit lower=-3.14159 upper=3.14159 effort=0.0 velocity=0.0

Commit message: quadruped created

File: body.urdf (robot description, URDF)
Before this commit: robot robot, 3 links, 2 joints
Links:
- added link BackLowerLeg, mass 1; collision box size=0.2 0.2 1; visual box size=0.2 0.2 1
- added link FrontLowerLeg, mass 1; collision box size=0.2 0.2 1; visual box size=0.2 0.2 1
- added link LeftLeg, mass 1; collision box size=1 0.2 0.2; visual box size=1 0.2 0.2
- added link LeftLowerLeg, mass 1; collision box size=0.2 0.2 1; visual box size=0.2 0.2 1
- added link RightLeg, mass 1; collision box size=1 0.2 0.2; visual box size=1 0.2 0.2
- added link RightLowerLeg, mass 1; collision box size=0.2 0.2 1; visual box size=0.2 0.2 1
- link BackLeg: geometry collision box size=0.2 1 0.2; visual box size=0.2 1 0.2
- link FrontLeg: geometry collision box size=0.2 1 0.2; visual box size=0.2 1 0.2
Joints:
- added joint BackLeg_BackLowerLeg: type revolute, parent BackLeg, child BackLowerLeg, origin xyz=0 -1 0 rpy=0 0 0, axis 1 0 0, limit lower=-3.14159 upper=3.14159 effort=0.0 velocity=0.0
- added joint FrontLeg_FrontLowerLeg: type revolute, parent FrontLeg, child FrontLowerLeg, origin xyz=0 1 0 rpy=0 0 0, axis 1 0 0, limit lower=-3.14159 upper=3.14159 effort=0.0 velocity=0.0
- added joint LeftLeg_LeftLowerLeg: type revolute, parent LeftLeg, child LeftLowerLeg, origin xyz=-1 0 0 rpy=0 0 0, axis 0 1 0, limit lower=-3.14159 upper=3.14159 effort=0.0 velocity=0.0
- added joint RightLeg_RightLowerLeg: type revolute, parent RightLeg, child RightLowerLeg, origin xyz=1 0 0 rpy=0 0 0, axis 0 1 0, limit lower=-3.14159 upper=3.14159 effort=0.0 velocity=0.0
- added joint Torso_LeftLeg: type revolute, parent Torso, child LeftLeg, origin xyz=-0.5 0 1 rpy=0 0 0, axis 0 1 0, limit lower=-3.14159 upper=3.14159 effort=0.0 velocity=0.0
- added joint Torso_RightLeg: type revolute, parent Torso, child RightLeg, origin xyz=0.5 0 1 rpy=0 0 0, axis 0 1 0, limit lower=-3.14159 upper=3.14159 effort=0.0 velocity=0.0
- joint Torso_BackLeg: axis 0 1 0 -> 1 0 0; origin xyz=-0.5 0 0.5 rpy=0 0 0 -> xyz=0 -0.5 1 rpy=0 0 0
- joint Torso_FrontLeg: axis 0 1 0 -> 1 0 0; origin xyz=0.5 0 0.5 rpy=0 0 0 -> xyz=0 0.5 1 rpy=0 0 0

Commit message: final_proj reddit

File: body.urdf (robot description, URDF)
Before this commit: robot robot, 9 links, 8 joints
Links:
- added link Antenna, mass 1; collision box size=0.1 2 0.1; visual box size=0.1 2 0.1
- added link Antenna2, mass 1; collision box size=0.1 0.1 3; visual box size=0.1 0.1 3
- link Torso: geometry collision box size=0.1 0.1 2; visual box size=0.1 0.1 2
Joints:
- added joint Antenna_Antenna2: type revolute, parent Antenna, child Antenna2, origin xyz=0 2 0 rpy=0 0 0, axis 1 0 0, limit lower=-3.14159 upper=3.14159 effort=0.0 velocity=0.0
- added joint Torso_Antenna: type revolute, parent Torso, child Antenna, origin xyz=0 0 3 rpy=0 0 0, axis 1 0 0, limit lower=-3.14159 upper=3.14159 effort=0.0 velocity=0.0
- joint BackLeg_BackLowerLeg: origin xyz=0 -1 0 rpy=0 0 0 -> xyz=0 -0.5 0 rpy=0 0 0
- joint FrontLeg_FrontLowerLeg: origin xyz=0 1 0 rpy=0 0 0 -> xyz=0 0.5 0 rpy=0 0 0
- joint LeftLeg_LeftLowerLeg: origin xyz=-1 0 0 rpy=0 0 0 -> xyz=-0.5 0 0 rpy=0 0 0
- joint RightLeg_RightLowerLeg: origin xyz=1 0 0 rpy=0 0 0 -> xyz=0.5 0 0 rpy=0 0 0
