Commit message: working on 1d morph

File: body0.urdf (robot description, URDF)
Before this commit: robot robot, 8 links, 7 joints
Links:
- added link Link10, mass 1; collision box size=0.2973082935680925 1.0141003756222573 0.4973516143947061; visual box size=0.2973082935680925 1.0141003756222573 0.4973516143947061
- added link Link11, mass 1; collision box size=0.9460634801152625 0.9942960409808996 0.728750621998889; visual box size=0.9460634801152625 0.9942960409808996 0.728750621998889
- added link Link9, mass 1; collision box size=1.04511916317611 1.2546525741670427 0.1994750599610103; visual box size=1.04511916317611 1.2546525741670427 0.1994750599610103
- link Link1: geometry collision box size=0.5531383102645525 1.1055304919101208 0.4105388232859567; visual box size=0.5531383102645525 1.1055304919101208 0.4105388232859567
- link Link2: geometry collision box size=0.4012971332457972 0.8298111935530137 0.2724769296097178; visual box size=0.4012971332457972 0.8298111935530137 0.2724769296097178
- link Link3: geometry collision box size=1.0438189118285521 1.0812838934696782 0.38741807424076236; visual box size=1.0438189118285521 1.0812838934696782 0.38741807424076236
- link Link4: geometry collision box size=0.14252406970109924 1.223359047005691 1.0353913912231092; visual box size=0.14252406970109924 1.223359047005691 1.0353913912231092
- link Link5: geometry collision box size=0.11832657264865323 0.3242083986461843 1.0359948186323953; visual box size=0.11832657264865323 0.3242083986461843 1.0359948186323953
- link Link6: geometry collision box size=1.0845625401215022 1.039661407082703 0.585743357899362; visual box size=1.0845625401215022 1.039661407082703 0.585743357899362
- link Link7: geometry collision box size=0.10179486915644723 0.3775038627636433 0.9598357700129521; visual box size=0.10179486915644723 0.3775038627636433 0.9598357700129521
- link Link8: geometry collision box size=0.26236032860442704 0.89180104326379 0.7974047352431408; visual box size=0.26236032860442704 0.89180104326379 0.7974047352431408
Joints:
- added joint Link10_Link11: type revolute, parent Link10, child Link11, origin xyz=0.2973082935680925 0 0 rpy=0 0 0, axis 0 1 0, limit lower=-3.14159 upper=3.14159 effort=0.0 velocity=0.0
- added joint Link8_Link9: type revolute, parent Link8, child Link9, origin xyz=0.26236032860442704 0 0 rpy=0 0 0, axis 0 1 0, limit lower=-3.14159 upper=3.14159 effort=0.0 velocity=0.0
- added joint Link9_Link10: type revolute, parent Link9, child Link10, origin xyz=1.04511916317611 0 0 rpy=0 0 0, axis 0 1 0, limit lower=-3.14159 upper=3.14159 effort=0.0 velocity=0.0
- joint Link1_Link2: origin xyz=0.3926152933911571 0 1 rpy=0 0 0 -> xyz=0.27656915513227626 0 1 rpy=0 0 0
- joint Link2_Link3: origin xyz=1.0328300499289045 0 0 rpy=0 0 0 -> xyz=0.4012971332457972 0 0 rpy=0 0 0
- joint Link3_Link4: origin xyz=0.6304640252001893 0 0 rpy=0 0 0 -> xyz=1.0438189118285521 0 0 rpy=0 0 0
- joint Link4_Link5: origin xyz=0.33479885559301825 0 0 rpy=0 0 0 -> xyz=0.14252406970109924 0 0 rpy=0 0 0
- joint Link5_Link6: origin xyz=0.5933132379308176 0 0 rpy=0 0 0 -> xyz=0.11832657264865323 0 0 rpy=0 0 0
- joint Link6_Link7: origin xyz=1.0868621347077214 0 0 rpy=0 0 0 -> xyz=1.0845625401215022 0 0 rpy=0 0 0
- joint Link7_Link8: origin xyz=1.0267997285226524 0 0 rpy=0 0 0 -> xyz=0.10179486915644723 0 0 rpy=0 0 0

File: body1.urdf (robot description, URDF)
Before this commit: robot robot, 6 links, 5 joints
Links:
- added link Link7, mass 1; collision box size=0.28408890612534754 1.229457524712727 0.8079511338063355; visual box size=0.28408890612534754 1.229457524712727 0.8079511338063355
- added link Link8, mass 1; collision box size=0.7214515669419528 0.4484919758941264 0.37599722964205506; visual box size=0.7214515669419528 0.4484919758941264 0.37599722964205506
- added link Link9, mass 1; collision box size=0.2608605929009815 0.9208792508884411 0.8895206522028694; visual box size=0.2608605929009815 0.9208792508884411 0.8895206522028694
- link Link1: geometry collision box size=0.7079826457515266 0.46947011901321606 0.9761772894300715; visual box size=0.7079826457515266 0.46947011901321606 0.9761772894300715
- link Link2: geometry collision box size=0.5582792482909972 1.2361189946250801 0.6391737500096384; visual box size=0.5582792482909972 1.2361189946250801 0.6391737500096384
- link Link3: geometry collision box size=0.19035434787250186 0.804634824835929 1.095795652044911; visual box size=0.19035434787250186 0.804634824835929 1.095795652044911
- link Link4: geometry collision box size=0.9554110208521306 0.4833442964892449 0.9844461014144263; visual box size=0.9554110208521306 0.4833442964892449 0.9844461014144263
- link Link5: geometry collision box size=0.27330062577852543 1.2115745840779883 0.9873255188209459; visual box size=0.27330062577852543 1.2115745840779883 0.9873255188209459
- link Link6: geometry collision box size=0.816716545303912 0.7835434899927445 0.9680322120327851; visual box size=0.816716545303912 0.7835434899927445 0.9680322120327851
Joints:
- added joint Link6_Link7: type revolute, parent Link6, child Link7, origin xyz=0.816716545303912 0 0 rpy=0 0 0, axis 0 1 0, limit lower=-3.14159 upper=3.14159 effort=0.0 velocity=0.0
- added joint Link7_Link8: type revolute, parent Link7, child Link8, origin xyz=0.28408890612534754 0 0 rpy=0 0 0, axis 0 1 0, limit lower=-3.14159 upper=3.14159 effort=0.0 velocity=0.0
- added joint Link8_Link9: type revolute, parent Link8, child Link9, origin xyz=0.7214515669419528 0 0 rpy=0 0 0, axis 0 1 0, limit lower=-3.14159 upper=3.14159 effort=0.0 velocity=0.0
- joint Link1_Link2: origin xyz=0.13478375262084424 0 1 rpy=0 0 0 -> xyz=0.3539913228757633 0 1 rpy=0 0 0
- joint Link2_Link3: origin xyz=0.5208985551470665 0 0 rpy=0 0 0 -> xyz=0.5582792482909972 0 0 rpy=0 0 0
- joint Link3_Link4: origin xyz=0.584183634812653 0 0 rpy=0 0 0 -> xyz=0.19035434787250186 0 0 rpy=0 0 0
- joint Link4_Link5: origin xyz=0.7277083612991726 0 0 rpy=0 0 0 -> xyz=0.9554110208521306 0 0 rpy=0 0 0
- joint Link5_Link6: origin xyz=0.5043995561689505 0 0 rpy=0 0 0 -> xyz=0.27330062577852543 0 0 rpy=0 0 0

File: body2.urdf (robot description, URDF)
Before this commit: robot robot, 10 links, 9 joints
Links:
- removed link Link10
- removed link Link8
- removed link Link9
- link Link1: geometry collision box size=0.7035279341604358 0.7831787016413974 1.067843941196919; visual box size=0.7035279341604358 0.7831787016413974 1.067843941196919
- link Link2: geometry collision box size=0.46586435976211227 0.96360009464071 0.7672040646501374; visual box size=0.46586435976211227 0.96360009464071 0.7672040646501374
- link Link3: geometry collision box size=0.8076453930425855 1.0529023954896204 0.9911899200501356; visual box size=0.8076453930425855 1.0529023954896204 0.9911899200501356
- link Link4: geometry collision box size=0.5222487917278587 1.2391053221852677 0.9589632168811043; visual box size=0.5222487917278587 1.2391053221852677 0.9589632168811043
- link Link5: geometry collision box size=0.8909374534273594 1.2814739462354583 0.5321955528947594; visual box size=0.8909374534273594 1.2814739462354583 0.5321955528947594
- link Link6: geometry collision box size=0.5593654725070155 1.0886511119227626 0.37504139550059024; visual box size=0.5593654725070155 1.0886511119227626 0.37504139550059024
- link Link7: geometry collision box size=0.6050980198488068 0.6753368428231754 0.9034075315610738; visual box size=0.6050980198488068 0.6753368428231754 0.9034075315610738
Joints:
- removed joint Link7_Link8
- removed joint Link8_Link9
- removed joint Link9_Link10
- joint Link1_Link2: origin xyz=0.3982782749902275 0 1 rpy=0 0 0 -> xyz=0.3517639670802179 0 1 rpy=0 0 0
- joint Link2_Link3: origin xyz=0.9137857309204861 0 0 rpy=0 0 0 -> xyz=0.46586435976211227 0 0 rpy=0 0 0
- joint Link3_Link4: origin xyz=0.727470240861943 0 0 rpy=0 0 0 -> xyz=0.8076453930425855 0 0 rpy=0 0 0
- joint Link4_Link5: origin xyz=0.18459151223833717 0 0 rpy=0 0 0 -> xyz=0.5222487917278587 0 0 rpy=0 0 0
- joint Link5_Link6: origin xyz=0.9204846762267082 0 0 rpy=0 0 0 -> xyz=0.8909374534273594 0 0 rpy=0 0 0
- joint Link6_Link7: origin xyz=0.7073545097694727 0 0 rpy=0 0 0 -> xyz=0.5593654725070155 0 0 rpy=0 0 0

File: body3.urdf (robot description, URDF)
Before this commit: robot robot, 7 links, 6 joints
Links:
- removed link Link6
- removed link Link7
- link Link1: geometry collision box size=0.5101798478472014 0.6713301289214575 0.9792001997808208; visual box size=0.5101798478472014 0.6713301289214575 0.9792001997808208
- link Link2: geometry collision box size=0.37532549174259056 0.4786979311987292 0.5937530677629886; visual box size=0.37532549174259056 0.4786979311987292 0.5937530677629886
- link Link3: geometry collision box size=0.515068403173107 0.754564367899738 0.21134186996902368; visual box size=0.515068403173107 0.754564367899738 0.21134186996902368
- link Link4: geometry collision box size=0.9895742219071145 0.40568009968797897 0.8080602702007883; visual box size=0.9895742219071145 0.40568009968797897 0.8080602702007883
- link Link5: geometry collision box size=1.0201737284573744 1.057697597585315 0.7651180601550257; visual box size=1.0201737284573744 1.057697597585315 0.7651180601550257
Joints:
- removed joint Link5_Link6
- removed joint Link6_Link7
- joint Link1_Link2: origin xyz=0.15378432348331023 0 1 rpy=0 0 0 -> xyz=0.2550899239236007 0 1 rpy=0 0 0
- joint Link2_Link3: origin xyz=0.6249473859774357 0 0 rpy=0 0 0 -> xyz=0.37532549174259056 0 0 rpy=0 0 0
- joint Link3_Link4: origin xyz=0.6819134822233387 0 0 rpy=0 0 0 -> xyz=0.515068403173107 0 0 rpy=0 0 0
- joint Link4_Link5: origin xyz=0.1964571071785798 0 0 rpy=0 0 0 -> xyz=0.9895742219071145 0 0 rpy=0 0 0

File: body4.urdf (robot description, URDF)
Before this commit: robot robot, 12 links, 11 joints
Links:
- link Link1: geometry collision box size=0.48450442849361 1.061420752325816 0.6067402691880247; visual box size=0.48450442849361 1.061420752325816 0.6067402691880247
- link Link10: geometry collision box size=0.6265829674842143 0.565470062073874 0.6912129602740407; visual box size=0.6265829674842143 0.565470062073874 0.6912129602740407
- link Link11: geometry collision box size=0.8131783266813847 0.737758598486215 0.6817185281909703; visual box size=0.8131783266813847 0.737758598486215 0.6817185281909703
- link Link12: geometry collision box size=0.9200891627837767 0.45934642391400465 0.5292636040404656; visual box size=0.9200891627837767 0.45934642391400465 0.5292636040404656
- link Link2: geometry collision box size=0.14825734994383635 0.9901328955951276 0.6291663739597234; visual box size=0.14825734994383635 0.9901328955951276 0.6291663739597234
- link Link3: geometry collision box size=0.7849262260781374 0.762720161158609 0.5560236095285491; visual box size=0.7849262260781374 0.762720161158609 0.5560236095285491
- link Link4: geometry collision box size=0.23459847233556022 0.3419739464438442 0.49517504625169406; visual box size=0.23459847233556022 0.3419739464438442 0.49517504625169406
- link Link5: geometry collision box size=0.48758153348978095 1.2725347358690648 0.5241556340610598; visual box size=0.48758153348978095 1.2725347358690648 0.5241556340610598
- link Link6: geometry collision box size=0.22210125747986034 0.877496863320619 0.9911395591832519; visual box size=0.22210125747986034 0.877496863320619 0.9911395591832519
- link Link7: geometry collision box size=0.6054718499820348 0.30522317792553494 0.7910010441093515; visual box size=0.6054718499820348 0.30522317792553494 0.7910010441093515
- link Link8: geometry collision box size=0.2792028023777663 1.0826532234041637 0.8428197830919844; visual box size=0.2792028023777663 1.0826532234041637 0.8428197830919844
- link Link9: geometry collision box size=0.2847091932221303 0.9916716182101319 0.1858818495323636; visual box size=0.2847091932221303 0.9916716182101319 0.1858818495323636
Joints:
- joint Link10_Link11: origin xyz=0.15658907256795798 0 0 rpy=0 0 0 -> xyz=0.6265829674842143 0 0 rpy=0 0 0
- joint Link11_Link12: origin xyz=0.6406922005933537 0 0 rpy=0 0 0 -> xyz=0.8131783266813847 0 0 rpy=0 0 0
- joint Link1_Link2: origin xyz=0.12152091413385253 0 1 rpy=0 0 0 -> xyz=0.242252214246805 0 1 rpy=0 0 0
- joint Link2_Link3: origin xyz=0.18950879210307361 0 0 rpy=0 0 0 -> xyz=0.14825734994383635 0 0 rpy=0 0 0
- joint Link3_Link4: origin xyz=1.0739662460319597 0 0 rpy=0 0 0 -> xyz=0.7849262260781374 0 0 rpy=0 0 0
- joint Link4_Link5: origin xyz=0.7060719003676633 0 0 rpy=0 0 0 -> xyz=0.23459847233556022 0 0 rpy=0 0 0
- joint Link5_Link6: origin xyz=0.4010796705287353 0 0 rpy=0 0 0 -> xyz=0.48758153348978095 0 0 rpy=0 0 0
- joint Link6_Link7: origin xyz=0.5678924892828824 0 0 rpy=0 0 0 -> xyz=0.22210125747986034 0 0 rpy=0 0 0
- joint Link7_Link8: origin xyz=1.0542006180336099 0 0 rpy=0 0 0 -> xyz=0.6054718499820348 0 0 rpy=0 0 0
- joint Link8_Link9: origin xyz=0.28383797546197986 0 0 rpy=0 0 0 -> xyz=0.2792028023777663 0 0 rpy=0 0 0
- joint Link9_Link10: origin xyz=0.27035401161648953 0 0 rpy=0 0 0 -> xyz=0.2847091932221303 0 0 rpy=0 0 0

File: body5.urdf (robot description, URDF)
Before this commit: robot robot, 7 links, 6 joints
Links:
- added link Link8, mass 1; collision box size=0.3123319136158116 0.8500081182409482 0.3504226672066504; visual box size=0.3123319136158116 0.8500081182409482 0.3504226672066504
- added link Link9, mass 1; collision box size=0.9890579203947528 0.6920092981073929 0.5287513275960938; visual box size=0.9890579203947528 0.6920092981073929 0.5287513275960938
- link Link1: geometry collision box size=0.19859659042551306 0.9344631143216107 0.5870877672155652; visual box size=0.19859659042551306 0.9344631143216107 0.5870877672155652
- link Link2: geometry collision box size=0.27266142605585786 0.41551374190648666 0.4106323132848151; visual box size=0.27266142605585786 0.41551374190648666 0.4106323132848151
- link Link3: geometry collision box size=0.6146928265210112 1.1303763310494335 0.6304025160468271; visual box size=0.6146928265210112 1.1303763310494335 0.6304025160468271
- link Link4: geometry collision box size=0.1310787326855817 0.5382148458804312 0.7625345484771695; visual box size=0.1310787326855817 0.5382148458804312 0.7625345484771695
- link Link5: geometry collision box size=0.9080995571585521 0.5924161693857528 1.0969411685080455; visual box size=0.9080995571585521 0.5924161693857528 1.0969411685080455
- link Link6: geometry collision box size=0.4143825607988574 1.013968174536492 0.3976212289723049; visual box size=0.4143825607988574 1.013968174536492 0.3976212289723049
- link Link7: geometry collision box size=0.3039417977933667 0.5657532254830715 0.3615994341755133; visual box size=0.3039417977933667 0.5657532254830715 0.3615994341755133
Joints:
- added joint Link7_Link8: type revolute, parent Link7, child Link8, origin xyz=0.3039417977933667 0 0 rpy=0 0 0, axis 0 1 0, limit lower=-3.14159 upper=3.14159 effort=0.0 velocity=0.0
- added joint Link8_Link9: type revolute, parent Link8, child Link9, origin xyz=0.3123319136158116 0 0 rpy=0 0 0, axis 0 1 0, limit lower=-3.14159 upper=3.14159 effort=0.0 velocity=0.0
- joint Link1_Link2: origin xyz=0.20563914182884746 0 1 rpy=0 0 0 -> xyz=0.09929829521275653 0 1 rpy=0 0 0
- joint Link2_Link3: origin xyz=0.9656949369613997 0 0 rpy=0 0 0 -> xyz=0.27266142605585786 0 0 rpy=0 0 0
- joint Link3_Link4: origin xyz=0.6204798975596879 0 0 rpy=0 0 0 -> xyz=0.6146928265210112 0 0 rpy=0 0 0
- joint Link4_Link5: origin xyz=0.16370788335109612 0 0 rpy=0 0 0 -> xyz=0.1310787326855817 0 0 rpy=0 0 0
- joint Link5_Link6: origin xyz=0.5742961683791459 0 0 rpy=0 0 0 -> xyz=0.9080995571585521 0 0 rpy=0 0 0
- joint Link6_Link7: origin xyz=0.8804402802847546 0 0 rpy=0 0 0 -> xyz=0.4143825607988574 0 0 rpy=0 0 0

File: body6.urdf (robot description, URDF)
Before this commit: robot robot, 9 links, 8 joints
Links:
- removed link Link6
- removed link Link7
- removed link Link8
- removed link Link9
- link Link1: geometry collision box size=0.7493290360791504 0.7376947410246597 0.6207971885796669; visual box size=0.7493290360791504 0.7376947410246597 0.6207971885796669
- link Link2: geometry collision box size=0.7426240867255934 0.47025981211196527 0.9377430442459271; visual box size=0.7426240867255934 0.47025981211196527 0.9377430442459271
- link Link3: geometry collision box size=0.5379379252500152 0.8324675018131422 1.022487379526909; visual box size=0.5379379252500152 0.8324675018131422 1.022487379526909
- link Link4: geometry collision box size=1.0822722799597173 1.0410374879080133 0.9387013225962182; visual box size=1.0822722799597173 1.0410374879080133 0.9387013225962182
- link Link5: geometry collision box size=0.9368934126168998 0.7368461114575036 0.5915594236340768; visual box size=0.9368934126168998 0.7368461114575036 0.5915594236340768
Joints:
- removed joint Link5_Link6
- removed joint Link6_Link7
- removed joint Link7_Link8
- removed joint Link8_Link9
- joint Link1_Link2: origin xyz=0.37969083700355966 0 1 rpy=0 0 0 -> xyz=0.3746645180395752 0 1 rpy=0 0 0
- joint Link2_Link3: origin xyz=1.0770445002662576 0 0 rpy=0 0 0 -> xyz=0.7426240867255934 0 0 rpy=0 0 0
- joint Link3_Link4: origin xyz=0.6931590843501994 0 0 rpy=0 0 0 -> xyz=0.5379379252500152 0 0 rpy=0 0 0
- joint Link4_Link5: origin xyz=0.6959229590538747 0 0 rpy=0 0 0 -> xyz=1.0822722799597173 0 0 rpy=0 0 0

File: body7.urdf (robot description, URDF)
Before this commit: robot robot, 8 links, 7 joints
Links:
- link Link1: geometry collision box size=0.5641837326907978 0.420744742027186 0.339945262295005; visual box size=0.5641837326907978 0.420744742027186 0.339945262295005
- link Link2: geometry collision box size=0.5412317143914053 1.1860208103753573 0.9376197101840035; visual box size=0.5412317143914053 1.1860208103753573 0.9376197101840035
- link Link3: geometry collision box size=0.6536152335266694 0.4185185986400493 0.9423754814077617; visual box size=0.6536152335266694 0.4185185986400493 0.9423754814077617
- link Link4: geometry collision box size=0.29005044689882 0.7612337181935458 0.5074874554602694; visual box size=0.29005044689882 0.7612337181935458 0.5074874554602694
- link Link5: geometry collision box size=0.7640655157278458 0.7318218241117513 0.6297240682256098; visual box size=0.7640655157278458 0.7318218241117513 0.6297240682256098
- link Link6: geometry collision box size=1.0359418521047563 0.9484335686051288 0.9778152620006713; visual box size=1.0359418521047563 0.9484335686051288 0.9778152620006713
- link Link7: geometry collision box size=1.0812507134372997 0.66569099759614 0.7736483760488954; visual box size=1.0812507134372997 0.66569099759614 0.7736483760488954
- link Link8: geometry collision box size=1.0919806781249528 0.39028745327145803 1.0135192897169565; visual box size=1.0919806781249528 0.39028745327145803 1.0135192897169565
Joints:
- joint Link1_Link2: origin xyz=0.4482109985508573 0 1 rpy=0 0 0 -> xyz=0.2820918663453989 0 1 rpy=0 0 0
- joint Link2_Link3: origin xyz=0.7130299998610368 0 0 rpy=0 0 0 -> xyz=0.5412317143914053 0 0 rpy=0 0 0
- joint Link3_Link4: origin xyz=1.0595052390167148 0 0 rpy=0 0 0 -> xyz=0.6536152335266694 0 0 rpy=0 0 0
- joint Link4_Link5: origin xyz=0.5210282558462116 0 0 rpy=0 0 0 -> xyz=0.29005044689882 0 0 rpy=0 0 0
- joint Link5_Link6: origin xyz=0.5493455370817377 0 0 rpy=0 0 0 -> xyz=0.7640655157278458 0 0 rpy=0 0 0
- joint Link6_Link7: origin xyz=0.6544463601836943 0 0 rpy=0 0 0 -> xyz=1.0359418521047563 0 0 rpy=0 0 0
- joint Link7_Link8: origin xyz=0.7193792682936345 0 0 rpy=0 0 0 -> xyz=1.0812507134372997 0 0 rpy=0 0 0

File: body8.urdf (robot description, URDF)
Before this commit: robot robot, 4 links, 3 joints
Links:
- added link Link5, mass 1; collision box size=0.8202511230708743 0.7225655707677043 0.22057293347953374; visual box size=0.8202511230708743 0.7225655707677043 0.22057293347953374
- added link Link6, mass 1; collision box size=0.3516327140482881 0.9192509289660642 1.1447470188020752; visual box size=0.3516327140482881 0.9192509289660642 1.1447470188020752
- added link Link7, mass 1; collision box size=0.6000914367263334 0.9903475248972704 0.18559345660846346; visual box size=0.6000914367263334 0.9903475248972704 0.18559345660846346
- link Link1: geometry collision box size=0.17786521510137968 0.6402421692334512 0.3956025789340343; visual box size=0.17786521510137968 0.6402421692334512 0.3956025789340343
- link Link2: geometry collision box size=0.4711755802546038 0.3284065487798254 0.9569221345577273; visual box size=0.4711755802546038 0.3284065487798254 0.9569221345577273
- link Link3: geometry collision box size=0.6944536185626146 0.6594403125923372 0.6377153627035025; visual box size=0.6944536185626146 0.6594403125923372 0.6377153627035025
- link Link4: geometry collision box size=0.4030212806114163 0.620159883325412 0.9107286853178014; visual box size=0.4030212806114163 0.620159883325412 0.9107286853178014
Joints:
- added joint Link4_Link5: type revolute, parent Link4, child Link5, origin xyz=0.4030212806114163 0 0 rpy=0 0 0, axis 0 1 0, limit lower=-3.14159 upper=3.14159 effort=0.0 velocity=0.0
- added joint Link5_Link6: type revolute, parent Link5, child Link6, origin xyz=0.8202511230708743 0 0 rpy=0 0 0, axis 0 1 0, limit lower=-3.14159 upper=3.14159 effort=0.0 velocity=0.0
- added joint Link6_Link7: type revolute, parent Link6, child Link7, origin xyz=0.3516327140482881 0 0 rpy=0 0 0, axis 0 1 0, limit lower=-3.14159 upper=3.14159 effort=0.0 velocity=0.0
- joint Link1_Link2: origin xyz=0.3621803581357074 0 1 rpy=0 0 0 -> xyz=0.08893260755068984 0 1 rpy=0 0 0
- joint Link2_Link3: origin xyz=0.4023262686352669 0 0 rpy=0 0 0 -> xyz=0.4711755802546038 0 0 rpy=0 0 0
- joint Link3_Link4: origin xyz=0.502761957999701 0 0 rpy=0 0 0 -> xyz=0.6944536185626146 0 0 rpy=0 0 0
