Commit message: working on 1d morph

File: body9.urdf (robot description, URDF)
Before this commit: robot robot, 9 links, 8 joints
Links:
- link Link1: geometry collision box size=0.4123414412955536 1.0986826017480504 0.4510019524369563; visual box size=0.4123414412955536 1.0986826017480504 0.4510019524369563
- link Link2: geometry collision box size=0.3023111962734326 1.2007186909929304 0.669887984662626; visual box size=0.3023111962734326 1.2007186909929304 0.669887984662626
- link Link3: geometry collision box size=0.33751983710293043 1.2160655397548885 1.1084411458375905; visual box size=0.33751983710293043 1.2160655397548885 1.1084411458375905
- link Link4: geometry collision box size=0.3898631275647386 0.38880529976492423 0.9868355824508108; visual box size=0.3898631275647386 0.38880529976492423 0.9868355824508108
- link Link5: geometry collision box size=0.12177138894682929 0.40134644607568976 0.17182901875665288; visual box size=0.12177138894682929 0.40134644607568976 0.17182901875665288
- link Link6: geometry collision box size=0.35536988828146787 0.3883231961401286 0.7589731858010853; visual box size=0.35536988828146787 0.3883231961401286 0.7589731858010853
- link Link7: geometry collision box size=0.4775230271915454 1.040547808011898 0.8955906855280195; visual box size=0.4775230271915454 1.040547808011898 0.8955906855280195
- link Link8: geometry collision box size=0.3512479307809774 0.8336973681626103 0.3870968062166935; visual box size=0.3512479307809774 0.8336973681626103 0.3870968062166935
- link Link9: geometry collision box size=0.1632026023747181 1.2372489435001557 0.971593799892134; visual box size=0.1632026023747181 1.2372489435001557 0.971593799892134
Joints:
- joint Link1_Link2: origin xyz=0.3592679059716981 0 1 rpy=0 0 0 -> xyz=0.2061707206477768 0 1 rpy=0 0 0
- joint Link2_Link3: origin xyz=0.11764033889678485 0 0 rpy=0 0 0 -> xyz=0.3023111962734326 0 0 rpy=0 0 0
- joint Link3_Link4: origin xyz=0.49344383564991234 0 0 rpy=0 0 0 -> xyz=0.33751983710293043 0 0 rpy=0 0 0
- joint Link4_Link5: origin xyz=0.6214269066044832 0 0 rpy=0 0 0 -> xyz=0.3898631275647386 0 0 rpy=0 0 0
- joint Link5_Link6: origin xyz=0.19726916953527265 0 0 rpy=0 0 0 -> xyz=0.12177138894682929 0 0 rpy=0 0 0
- joint Link6_Link7: origin xyz=0.4929041653773416 0 0 rpy=0 0 0 -> xyz=0.35536988828146787 0 0 rpy=0 0 0
- joint Link7_Link8: origin xyz=0.29388213877117286 0 0 rpy=0 0 0 -> xyz=0.4775230271915454 0 0 rpy=0 0 0
- joint Link8_Link9: origin xyz=0.1401697213566622 0 0 rpy=0 0 0 -> xyz=0.3512479307809774 0 0 rpy=0 0 0

Commit message: morpholies generate, fitness not working

File: body0.urdf (robot description, URDF)
Before this commit: robot robot, 11 links, 10 joints
Links:
- removed link Link11
- link Link1: geometry collision box size=0.3073689814468461 0.6960708610924271 0.9285824049199852; visual box size=0.3073689814468461 0.6960708610924271 0.9285824049199852
- link Link10: geometry collision box size=0.35716249430598623 0.4526664716612497 1.01778815896125; visual box size=0.35716249430598623 0.4526664716612497 1.01778815896125
- link Link2: geometry collision box size=0.43991558639617745 0.9241634215918211 0.18357688866008567; visual box size=0.43991558639617745 0.9241634215918211 0.18357688866008567
- link Link3: geometry collision box size=0.9290351203387004 1.263233249369133 0.680159960759653; visual box size=0.9290351203387004 1.263233249369133 0.680159960759653
- link Link4: geometry collision box size=0.4287130340033498 0.39871469932763387 0.46870977473952435; visual box size=0.4287130340033498 0.39871469932763387 0.46870977473952435
- link Link5: geometry collision box size=0.8536572173733947 0.8060800830227222 0.44211657050038644; visual box size=0.8536572173733947 0.8060800830227222 0.44211657050038644
- link Link6: geometry collision box size=0.4297001311230245 0.37206583606003446 0.8697084355181331; visual box size=0.4297001311230245 0.37206583606003446 0.8697084355181331
- link Link7: geometry collision box size=0.5732518551937431 0.5564827016741087 0.6810518353385254; visual box size=0.5732518551937431 0.5564827016741087 0.6810518353385254
- link Link8: geometry collision box size=0.7364418168913789 0.6038377089482236 0.24179835640038913; visual box size=0.7364418168913789 0.6038377089482236 0.24179835640038913
- link Link9: geometry collision box size=0.5415490349364924 0.7968626441497395 0.4048986469148096; visual box size=0.5415490349364924 0.7968626441497395 0.4048986469148096
Joints:
- removed joint Link10_Link11
- joint Link1_Link2: origin xyz=0.27656915513227626 0 1 rpy=0 0 0 -> xyz=0.15368449072342305 0 1 rpy=0 0 0
- joint Link2_Link3: origin xyz=0.4012971332457972 0 0 rpy=0 0 0 -> xyz=0.43991558639617745 0 0 rpy=0 0 0
- joint Link3_Link4: origin xyz=1.0438189118285521 0 0 rpy=0 0 0 -> xyz=0.9290351203387004 0 0 rpy=0 0 0
- joint Link4_Link5: origin xyz=0.14252406970109924 0 0 rpy=0 0 0 -> xyz=0.4287130340033498 0 0 rpy=0 0 0
- joint Link5_Link6: origin xyz=0.11832657264865323 0 0 rpy=0 0 0 -> xyz=0.8536572173733947 0 0 rpy=0 0 0
- joint Link6_Link7: origin xyz=1.0845625401215022 0 0 rpy=0 0 0 -> xyz=0.4297001311230245 0 0 rpy=0 0 0
- joint Link7_Link8: origin xyz=0.10179486915644723 0 0 rpy=0 0 0 -> xyz=0.5732518551937431 0 0 rpy=0 0 0
- joint Link8_Link9: origin xyz=0.26236032860442704 0 0 rpy=0 0 0 -> xyz=0.7364418168913789 0 0 rpy=0 0 0
- joint Link9_Link10: origin xyz=1.04511916317611 0 0 rpy=0 0 0 -> xyz=0.5415490349364924 0 0 rpy=0 0 0

File: body1.urdf (robot description, URDF)
Before this commit: robot robot, 9 links, 8 joints
Links:
- removed link Link8
- removed link Link9
- link Link1: geometry collision box size=0.12467758133856757 0.3134571697207981 0.3560222425944144; visual box size=0.12467758133856757 0.3134571697207981 0.3560222425944144
- link Link2: geometry collision box size=0.559731590487421 1.1816663299770025 0.7270062518582279; visual box size=0.559731590487421 1.1816663299770025 0.7270062518582279
- link Link3: geometry collision box size=0.2755342325951592 0.5747287088885535 0.2580200066490802; visual box size=0.2755342325951592 0.5747287088885535 0.2580200066490802
- link Link4: geometry collision box size=0.8971704145220685 0.7329805749575133 0.2701759808191292; visual box size=0.8971704145220685 0.7329805749575133 0.2701759808191292
- link Link5: geometry collision box size=0.5785943848866345 0.38323539176070126 0.4843961909867184; visual box size=0.5785943848866345 0.38323539176070126 0.4843961909867184
- link Link6: geometry collision box size=0.7809623628830878 0.8952407918309835 0.36011495279156136; visual box size=0.7809623628830878 0.8952407918309835 0.36011495279156136
- link Link7: geometry collision box size=0.9797643233988137 0.814745614866283 0.9894597208773402; visual box size=0.9797643233988137 0.814745614866283 0.9894597208773402
Joints:
- removed joint Link7_Link8
- removed joint Link8_Link9
- joint Link1_Link2: origin xyz=0.3539913228757633 0 1 rpy=0 0 0 -> xyz=0.062338790669283786 0 1 rpy=0 0 0
- joint Link2_Link3: origin xyz=0.5582792482909972 0 0 rpy=0 0 0 -> xyz=0.559731590487421 0 0 rpy=0 0 0
- joint Link3_Link4: origin xyz=0.19035434787250186 0 0 rpy=0 0 0 -> xyz=0.2755342325951592 0 0 rpy=0 0 0
- joint Link4_Link5: origin xyz=0.9554110208521306 0 0 rpy=0 0 0 -> xyz=0.8971704145220685 0 0 rpy=0 0 0
- joint Link5_Link6: origin xyz=0.27330062577852543 0 0 rpy=0 0 0 -> xyz=0.5785943848866345 0 0 rpy=0 0 0
- joint Link6_Link7: origin xyz=0.816716545303912 0 0 rpy=0 0 0 -> xyz=0.7809623628830878 0 0 rpy=0 0 0

File: body2.urdf (robot description, URDF)
Before this commit: robot robot, 7 links, 6 joints
Links:
- removed link Link4
- removed link Link5
- removed link Link6
- removed link Link7
- link Link1: geometry collision box size=0.10796532072030854 0.9529575625368143 0.644786351688626; visual box size=0.10796532072030854 0.9529575625368143 0.644786351688626
- link Link2: geometry collision box size=0.6394041496064782 0.6404785154411667 0.7261689807880379; visual box size=0.6394041496064782 0.6404785154411667 0.7261689807880379
- link Link3: geometry collision box size=0.9825328908185761 1.195123018175701 0.31793409662069727; visual box size=0.9825328908185761 1.195123018175701 0.31793409662069727
Joints:
- removed joint Link3_Link4
- removed joint Link4_Link5
- removed joint Link5_Link6
- removed joint Link6_Link7
- joint Link1_Link2: origin xyz=0.3517639670802179 0 1 rpy=0 0 0 -> xyz=0.05398266036015427 0 1 rpy=0 0 0
- joint Link2_Link3: origin xyz=0.46586435976211227 0 0 rpy=0 0 0 -> xyz=0.6394041496064782 0 0 rpy=0 0 0

File: body3.urdf (robot description, URDF)
Before this commit: robot robot, 5 links, 4 joints
Links:
- added link Link10, mass 1; collision box size=0.4054657986418473 0.885913578861192 0.20716463425759132; visual box size=0.4054657986418473 0.885913578861192 0.20716463425759132
- added link Link11, mass 1; collision box size=0.35135997172967404 0.8619300412594448 0.5340194170964191; visual box size=0.35135997172967404 0.8619300412594448 0.5340194170964191
- added link Link12, mass 1; collision box size=0.9362445507161601 0.9503096122202455 0.3247088511220829; visual box size=0.9362445507161601 0.9503096122202455 0.3247088511220829
- added link Link6, mass 1; collision box size=0.8459720065221463 1.171514335961502 0.5312913577229388; visual box size=0.8459720065221463 1.171514335961502 0.5312913577229388
- added link Link7, mass 1; collision box size=1.0267569850322114 1.1499362890192004 0.18063246592085322; visual box size=1.0267569850322114 1.1499362890192004 0.18063246592085322
- added link Link8, mass 1; collision box size=0.9997592710129654 0.9841141516991709 0.3801669972397157; visual box size=0.9997592710129654 0.9841141516991709 0.3801669972397157
- added link Link9, mass 1; collision box size=0.3329142505644618 1.1094736001765988 0.46420971411971024; visual box size=0.3329142505644618 1.1094736001765988 0.46420971411971024
- link Link1: geometry collision box size=0.10139518170512277 0.5613071257332158 0.4488724409499115; visual box size=0.10139518170512277 0.5613071257332158 0.4488724409499115
- link Link2: geometry collision box size=0.9643274715001173 1.0833199775460418 0.37703299548141445; visual box size=0.9643274715001173 1.0833199775460418 0.37703299548141445
- link Link3: geometry collision box size=0.5472093584333912 0.44519284151062893 0.9961936419367675; visual box size=0.5472093584333912 0.44519284151062893 0.9961936419367675
- link Link4: geometry collision box size=0.2364828286039863 0.3317962016655445 0.49761956757701653; visual box size=0.2364828286039863 0.3317962016655445 0.49761956757701653
- link Link5: geometry collision box size=0.5341970686804387 1.012464537767206 0.18849141307293524; visual box size=0.5341970686804387 1.012464537767206 0.18849141307293524
Joints:
- added joint Link10_Link11: type revolute, parent Link10, child Link11, origin xyz=0.4054657986418473 0 0 rpy=0 0 0, axis 0 1 0, limit lower=-3.14159 upper=3.14159 effort=0.0 velocity=0.0
- added joint Link11_Link12: type revolute, parent Link11, child Link12, origin xyz=0.35135997172967404 0 0 rpy=0 0 0, axis 0 1 0, limit lower=-3.14159 upper=3.14159 effort=0.0 velocity=0.0
- added joint Link5_Link6: type revolute, parent Link5, child Link6, origin xyz=0.5341970686804387 0 0 rpy=0 0 0, axis 0 1 0, limit lower=-3.14159 upper=3.14159 effort=0.0 velocity=0.0
- added joint Link6_Link7: type revolute, parent Link6, child Link7, origin xyz=0.8459720065221463 0 0 rpy=0 0 0, axis 0 1 0, limit lower=-3.14159 upper=3.14159 effort=0.0 velocity=0.0
- added joint Link7_Link8: type revolute, parent Link7, child Link8, origin xyz=1.0267569850322114 0 0 rpy=0 0 0, axis 0 1 0, limit lower=-3.14159 upper=3.14159 effort=0.0 velocity=0.0
- added joint Link8_Link9: type revolute, parent Link8, child Link9, origin xyz=0.9997592710129654 0 0 rpy=0 0 0, axis 0 1 0, limit lower=-3.14159 upper=3.14159 effort=0.0 velocity=0.0
- added joint Link9_Link10: type revolute, parent Link9, child Link10, origin xyz=0.3329142505644618 0 0 rpy=0 0 0, axis 0 1 0, limit lower=-3.14159 upper=3.14159 effort=0.0 velocity=0.0
- joint Link1_Link2: origin xyz=0.2550899239236007 0 1 rpy=0 0 0 -> xyz=0.05069759085256138 0 1 rpy=0 0 0
- joint Link2_Link3: origin xyz=0.37532549174259056 0 0 rpy=0 0 0 -> xyz=0.9643274715001173 0 0 rpy=0 0 0
- joint Link3_Link4: origin xyz=0.515068403173107 0 0 rpy=0 0 0 -> xyz=0.5472093584333912 0 0 rpy=0 0 0
- joint Link4_Link5: origin xyz=0.9895742219071145 0 0 rpy=0 0 0 -> xyz=0.2364828286039863 0 0 rpy=0 0 0

File: body4.urdf (robot description, URDF)
Before this commit: robot robot, 12 links, 11 joints
Links:
- removed link Link10
- removed link Link11
- removed link Link12
- removed link Link8
- removed link Link9
- link Link1: geometry collision box size=0.678311392789938 1.0680802045400577 0.15152197481961735; visual box size=0.678311392789938 1.0680802045400577 0.15152197481961735
- link Link2: geometry collision box size=0.9207417253949284 0.5655409520012191 0.34247465223231943; visual box size=0.9207417253949284 0.5655409520012191 0.34247465223231943
- link Link3: geometry collision box size=0.25103412870295383 1.1516158398472782 0.5590280463941075; visual box size=0.25103412870295383 1.1516158398472782 0.5590280463941075
- link Link4: geometry collision box size=0.5122412435084318 1.2014899679763795 0.28767120952196124; visual box size=0.5122412435084318 1.2014899679763795 0.28767120952196124
- link Link5: geometry collision box size=0.9836713545861838 0.6552106145743051 0.31477386180359546; visual box size=0.9836713545861838 0.6552106145743051 0.31477386180359546
- link Link6: geometry collision box size=0.14819106903355342 0.8498914469873255 0.9276884173223877; visual box size=0.14819106903355342 0.8498914469873255 0.9276884173223877
- link Link7: geometry collision box size=0.3596348132634978 0.5861285334974737 1.098811033989789; visual box size=0.3596348132634978 0.5861285334974737 1.098811033989789
Joints:
- removed joint Link10_Link11
- removed joint Link11_Link12
- removed joint Link7_Link8
- removed joint Link8_Link9
- removed joint Link9_Link10
- joint Link1_Link2: origin xyz=0.242252214246805 0 1 rpy=0 0 0 -> xyz=0.339155696394969 0 1 rpy=0 0 0
- joint Link2_Link3: origin xyz=0.14825734994383635 0 0 rpy=0 0 0 -> xyz=0.9207417253949284 0 0 rpy=0 0 0
- joint Link3_Link4: origin xyz=0.7849262260781374 0 0 rpy=0 0 0 -> xyz=0.25103412870295383 0 0 rpy=0 0 0
- joint Link4_Link5: origin xyz=0.23459847233556022 0 0 rpy=0 0 0 -> xyz=0.5122412435084318 0 0 rpy=0 0 0
- joint Link5_Link6: origin xyz=0.48758153348978095 0 0 rpy=0 0 0 -> xyz=0.9836713545861838 0 0 rpy=0 0 0
- joint Link6_Link7: origin xyz=0.22210125747986034 0 0 rpy=0 0 0 -> xyz=0.14819106903355342 0 0 rpy=0 0 0
