Commit message: done

File: body0.urdf (robot description, URDF)
Before this commit: robot robot, 10 links, 9 joints
Links:
- link Link1: geometry collision box size=0.3858553328787403 1.005416844744965 0.6134885098239043; visual box size=0.3858553328787403 1.005416844744965 0.6134885098239043
- link Link10: geometry collision box size=0.748981289062618 0.47408813906070574 0.7205976913733734; visual box size=0.748981289062618 0.47408813906070574 0.7205976913733734
- link Link2: geometry collision box size=1.0713668230413884 0.7825686570955968 1.0855603629587676; visual box size=1.0713668230413884 0.7825686570955968 1.0855603629587676
- link Link3: geometry collision box size=1.0119438504694291 0.7741020143623136 0.610663916423267; visual box size=1.0119438504694291 0.7741020143623136 0.610663916423267
- link Link4: geometry collision box size=1.0688683422390406 1.2027582914880677 0.6015580091941642; visual box size=1.0688683422390406 1.2027582914880677 0.6015580091941642
- link Link5: geometry collision box size=0.5612359157856884 0.7503193659987777 0.3074327751550274; visual box size=0.5612359157856884 0.7503193659987777 0.3074327751550274
- link Link6: geometry collision box size=0.8975985837948535 0.7109941892927216 0.6361765981305872; visual box size=0.8975985837948535 0.7109941892927216 0.6361765981305872
- link Link7: geometry collision box size=0.7737150683185089 0.4493182034756114 0.5937685842143434; visual box size=0.7737150683185089 0.4493182034756114 0.5937685842143434
- link Link8: geometry collision box size=1.006834561141499 0.7787271680015022 0.9902872757741942; visual box size=1.006834561141499 0.7787271680015022 0.9902872757741942
- link Link9: geometry collision box size=0.8192968401973321 1.1657966514995264 0.3439364336135313; visual box size=0.8192968401973321 1.1657966514995264 0.3439364336135313
Joints:
- joint Link1_Link2: origin xyz=0.15368449072342305 0 1 rpy=0 0 0 -> xyz=0.19292766643937015 0 1 rpy=0 0 0
- joint Link2_Link3: origin xyz=0.43991558639617745 0 0 rpy=0 0 0 -> xyz=1.0713668230413884 0 0 rpy=0 0 0
- joint Link3_Link4: origin xyz=0.9290351203387004 0 0 rpy=0 0 0 -> xyz=1.0119438504694291 0 0 rpy=0 0 0
- joint Link4_Link5: origin xyz=0.4287130340033498 0 0 rpy=0 0 0 -> xyz=1.0688683422390406 0 0 rpy=0 0 0
- joint Link5_Link6: origin xyz=0.8536572173733947 0 0 rpy=0 0 0 -> xyz=0.5612359157856884 0 0 rpy=0 0 0
- joint Link6_Link7: origin xyz=0.4297001311230245 0 0 rpy=0 0 0 -> xyz=0.8975985837948535 0 0 rpy=0 0 0
- joint Link7_Link8: origin xyz=0.5732518551937431 0 0 rpy=0 0 0 -> xyz=0.7737150683185089 0 0 rpy=0 0 0
- joint Link8_Link9: origin xyz=0.7364418168913789 0 0 rpy=0 0 0 -> xyz=1.006834561141499 0 0 rpy=0 0 0
- joint Link9_Link10: origin xyz=0.5415490349364924 0 0 rpy=0 0 0 -> xyz=0.8192968401973321 0 0 rpy=0 0 0

File: body1.urdf (robot description, URDF)
Before this commit: robot robot, 7 links, 6 joints
Links:
- added link Link8, mass 1; collision box size=0.2574560196057142 1.061820910661041 0.2771369961707181; visual box size=0.2574560196057142 1.061820910661041 0.2771369961707181
- added link Link9, mass 1; collision box size=0.5380670816978914 1.0335717546314362 1.0955730053929205; visual box size=0.5380670816978914 1.0335717546314362 1.0955730053929205
- link Link1: geometry collision box size=0.20421575839048747 0.4011373363289788 0.5870949387437239; visual box size=0.20421575839048747 0.4011373363289788 0.5870949387437239
- link Link2: geometry collision box size=0.5164588930811218 0.7581857896674835 0.18406744478619982; visual box size=0.5164588930811218 0.7581857896674835 0.18406744478619982
- link Link3: geometry collision box size=0.8833262706192718 0.3808799065733807 0.9569770994029764; visual box size=0.8833262706192718 0.3808799065733807 0.9569770994029764
- link Link4: geometry collision box size=0.3315467823120757 0.6682204793979023 0.3671324235626998; visual box size=0.3315467823120757 0.6682204793979023 0.3671324235626998
- link Link5: geometry collision box size=0.49402756202223086 0.9769205638942056 0.1653981419237017; visual box size=0.49402756202223086 0.9769205638942056 0.1653981419237017
- link Link6: geometry collision box size=0.8952719306418322 0.772460027383842 0.3111628362275507; visual box size=0.8952719306418322 0.772460027383842 0.3111628362275507
- link Link7: geometry collision box size=0.32753401020537765 0.992786735286153 1.0449073758904264; visual box size=0.32753401020537765 0.992786735286153 1.0449073758904264
Joints:
- added joint Link7_Link8: type revolute, parent Link7, child Link8, origin xyz=0.32753401020537765 0 0 rpy=0 0 0, axis 0 1 0, limit lower=-3.14159 upper=3.14159 effort=0.0 velocity=0.0
- added joint Link8_Link9: type revolute, parent Link8, child Link9, origin xyz=0.2574560196057142 0 0 rpy=0 0 0, axis 0 1 0, limit lower=-3.14159 upper=3.14159 effort=0.0 velocity=0.0
- joint Link1_Link2: origin xyz=0.062338790669283786 0 1 rpy=0 0 0 -> xyz=0.10210787919524374 0 1 rpy=0 0 0
- joint Link2_Link3: origin xyz=0.559731590487421 0 0 rpy=0 0 0 -> xyz=0.5164588930811218 0 0 rpy=0 0 0
- joint Link3_Link4: origin xyz=0.2755342325951592 0 0 rpy=0 0 0 -> xyz=0.8833262706192718 0 0 rpy=0 0 0
- joint Link4_Link5: origin xyz=0.8971704145220685 0 0 rpy=0 0 0 -> xyz=0.3315467823120757 0 0 rpy=0 0 0
- joint Link5_Link6: origin xyz=0.5785943848866345 0 0 rpy=0 0 0 -> xyz=0.49402756202223086 0 0 rpy=0 0 0
- joint Link6_Link7: origin xyz=0.7809623628830878 0 0 rpy=0 0 0 -> xyz=0.8952719306418322 0 0 rpy=0 0 0

File: body2.urdf (robot description, URDF)
Before this commit: robot robot, 3 links, 2 joints
Links:
- added link Link10, mass 1; collision box size=0.6563170306710877 0.5277364250540628 0.32962899385706723; visual box size=0.6563170306710877 0.5277364250540628 0.32962899385706723
- added link Link11, mass 1; collision box size=0.530152421299476 0.7795520538136917 0.8219613771397162; visual box size=0.530152421299476 0.7795520538136917 0.8219613771397162
- added link Link12, mass 1; collision box size=0.6895106608372885 0.34240923462871836 0.27222011515911904; visual box size=0.6895106608372885 0.34240923462871836 0.27222011515911904
- added link Link4, mass 1; collision box size=0.3298802349316594 0.9326802413463651 0.5268764214406144; visual box size=0.3298802349316594 0.9326802413463651 0.5268764214406144
- added link Link5, mass 1; collision box size=0.9075250993279642 0.8123594781745374 0.3747836801220247; visual box size=0.9075250993279642 0.8123594781745374 0.3747836801220247
- added link Link6, mass 1; collision box size=0.9765111556423784 0.9185559617759689 0.7946791449527137; visual box size=0.9765111556423784 0.9185559617759689 0.7946791449527137
- added link Link7, mass 1; collision box size=0.14228066732264935 1.0880508784653664 1.0397730564731027; visual box size=0.14228066732264935 1.0880508784653664 1.0397730564731027
- added link Link8, mass 1; collision box size=0.5071773706300138 0.47902956240824796 0.2145665366498348; visual box size=0.5071773706300138 0.47902956240824796 0.2145665366498348
- added link Link9, mass 1; collision box size=0.39029303910840696 0.6132526239589229 0.482108287938551; visual box size=0.39029303910840696 0.6132526239589229 0.482108287938551
- link Link1: geometry collision box size=0.8181800074109267 0.36247904288367777 1.0305964117364728; visual box size=0.8181800074109267 0.36247904288367777 1.0305964117364728
- link Link2: geometry collision box size=0.7923590534502866 0.9477558148998664 1.1333155746103534; visual box size=0.7923590534502866 0.9477558148998664 1.1333155746103534
- link Link3: geometry collision box size=0.7533849456709687 0.5045595778541412 0.8518544601240516; visual box size=0.7533849456709687 0.5045595778541412 0.8518544601240516
Joints:
- added joint Link10_Link11: type revolute, parent Link10, child Link11, origin xyz=0.6563170306710877 0 0 rpy=0 0 0, axis 0 1 0, limit lower=-3.14159 upper=3.14159 effort=0.0 velocity=0.0
- added joint Link11_Link12: type revolute, parent Link11, child Link12, origin xyz=0.530152421299476 0 0 rpy=0 0 0, axis 0 1 0, limit lower=-3.14159 upper=3.14159 effort=0.0 velocity=0.0
- added joint Link3_Link4: type revolute, parent Link3, child Link4, origin xyz=0.7533849456709687 0 0 rpy=0 0 0, axis 0 1 0, limit lower=-3.14159 upper=3.14159 effort=0.0 velocity=0.0
- added joint Link4_Link5: type revolute, parent Link4, child Link5, origin xyz=0.3298802349316594 0 0 rpy=0 0 0, axis 0 1 0, limit lower=-3.14159 upper=3.14159 effort=0.0 velocity=0.0
- added joint Link5_Link6: type revolute, parent Link5, child Link6, origin xyz=0.9075250993279642 0 0 rpy=0 0 0, axis 0 1 0, limit lower=-3.14159 upper=3.14159 effort=0.0 velocity=0.0
- added joint Link6_Link7: type revolute, parent Link6, child Link7, origin xyz=0.9765111556423784 0 0 rpy=0 0 0, axis 0 1 0, limit lower=-3.14159 upper=3.14159 effort=0.0 velocity=0.0
- added joint Link7_Link8: type revolute, parent Link7, child Link8, origin xyz=0.14228066732264935 0 0 rpy=0 0 0, axis 0 1 0, limit lower=-3.14159 upper=3.14159 effort=0.0 velocity=0.0
- added joint Link8_Link9: type revolute, parent Link8, child Link9, origin xyz=0.5071773706300138 0 0 rpy=0 0 0, axis 0 1 0, limit lower=-3.14159 upper=3.14159 effort=0.0 velocity=0.0
- added joint Link9_Link10: type revolute, parent Link9, child Link10, origin xyz=0.39029303910840696 0 0 rpy=0 0 0, axis 0 1 0, limit lower=-3.14159 upper=3.14159 effort=0.0 velocity=0.0
- joint Link1_Link2: origin xyz=0.05398266036015427 0 1 rpy=0 0 0 -> xyz=0.40909000370546333 0 1 rpy=0 0 0
- joint Link2_Link3: origin xyz=0.6394041496064782 0 0 rpy=0 0 0 -> xyz=0.7923590534502866 0 0 rpy=0 0 0

File: body3.urdf (robot description, URDF)
Before this commit: robot robot, 12 links, 11 joints
Links:
- removed link Link10
- removed link Link11
- removed link Link12
- removed link Link4
- removed link Link5
- removed link Link6
- removed link Link7
- removed link Link8
- removed link Link9
- link Link1: geometry collision box size=1.0870468303900616 0.7599848832683025 0.6736167588100569; visual box size=1.0870468303900616 0.7599848832683025 0.6736167588100569
- link Link2: geometry collision box size=0.3715316684299145 0.6023718708272869 0.5189273280257871; visual box size=0.3715316684299145 0.6023718708272869 0.5189273280257871
- link Link3: geometry collision box size=1.0442469783421418 0.5016291939885877 0.8610383819127854; visual box size=1.0442469783421418 0.5016291939885877 0.8610383819127854
Joints:
- removed joint Link10_Link11
- removed joint Link11_Link12
- removed joint Link3_Link4
- removed joint Link4_Link5
- removed joint Link5_Link6
- removed joint Link6_Link7
- removed joint Link7_Link8
- removed joint Link8_Link9
- removed joint Link9_Link10
- joint Link1_Link2: origin xyz=0.05069759085256138 0 1 rpy=0 0 0 -> xyz=0.5435234151950308 0 1 rpy=0 0 0
- joint Link2_Link3: origin xyz=0.9643274715001173 0 0 rpy=0 0 0 -> xyz=0.3715316684299145 0 0 rpy=0 0 0

File: body4.urdf (robot description, URDF)
Before this commit: robot robot, 7 links, 6 joints
Links:
- link Link1: geometry collision box size=0.3430361629932399 1.0922102890134489 1.043083911009194; visual box size=0.3430361629932399 1.0922102890134489 1.043083911009194
- link Link2: geometry collision box size=0.8380803891788293 0.7518883469375663 0.9793717020585966; visual box size=0.8380803891788293 0.7518883469375663 0.9793717020585966
- link Link3: geometry collision box size=0.238653574247247 1.2702192253999824 0.7996229835930605; visual box size=0.238653574247247 1.2702192253999824 0.7996229835930605
- link Link4: geometry collision box size=0.8496985649243783 1.1679098523298372 0.25374950115612027; visual box size=0.8496985649243783 1.1679098523298372 0.25374950115612027
- link Link5: geometry collision box size=0.39031000932257554 1.0100218661752456 1.010407414086039; visual box size=0.39031000932257554 1.0100218661752456 1.010407414086039
- link Link6: geometry collision box size=0.357688454730666 0.40498292912608863 0.39912906170598195; visual box size=0.357688454730666 0.40498292912608863 0.39912906170598195
- link Link7: geometry collision box size=0.1321164077999242 0.32702948619525524 1.0792640165504532; visual box size=0.1321164077999242 0.32702948619525524 1.0792640165504532
Joints:
- joint Link1_Link2: origin xyz=0.339155696394969 0 1 rpy=0 0 0 -> xyz=0.17151808149661996 0 1 rpy=0 0 0
- joint Link2_Link3: origin xyz=0.9207417253949284 0 0 rpy=0 0 0 -> xyz=0.8380803891788293 0 0 rpy=0 0 0
- joint Link3_Link4: origin xyz=0.25103412870295383 0 0 rpy=0 0 0 -> xyz=0.238653574247247 0 0 rpy=0 0 0
- joint Link4_Link5: origin xyz=0.5122412435084318 0 0 rpy=0 0 0 -> xyz=0.8496985649243783 0 0 rpy=0 0 0
- joint Link5_Link6: origin xyz=0.9836713545861838 0 0 rpy=0 0 0 -> xyz=0.39031000932257554 0 0 rpy=0 0 0
- joint Link6_Link7: origin xyz=0.14819106903355342 0 0 rpy=0 0 0 -> xyz=0.357688454730666 0 0 rpy=0 0 0
