Commit message: couple changes, rm body

File: body0.urdf (robot description, URDF)
Before this commit: robot robot, 10 links, 9 joints
Links:
- removed link Link10
- removed link Link7
- removed link Link8
- removed link Link9
- link Link1: geometry collision box size=0.5924397612754916 0.6217148535450534 0.9864050424687; visual box size=0.5924397612754916 0.6217148535450534 0.9864050424687
- link Link2: geometry collision box size=0.5765937489915485 1.1974399088284298 1.0872535459500814; visual box size=0.5765937489915485 1.1974399088284298 1.0872535459500814
- link Link3: geometry collision box size=0.29048986510979236 0.7041291136919599 0.279384418174912; visual box size=0.29048986510979236 0.7041291136919599 0.279384418174912
- link Link4: geometry collision box size=0.6305169742925424 0.9678171384608216 1.0104849464825363; visual box size=0.6305169742925424 0.9678171384608216 1.0104849464825363
- link Link5: geometry collision box size=0.8361367164541827 0.409757270037628 0.5188195745881915; visual box size=0.8361367164541827 0.409757270037628 0.5188195745881915
- link Link6: geometry collision box size=0.5193492398115318 0.9239998293089662 0.20364922557178486; visual box size=0.5193492398115318 0.9239998293089662 0.20364922557178486
Joints:
- removed joint Link6_Link7
- removed joint Link7_Link8
- removed joint Link8_Link9
- removed joint Link9_Link10
- joint Link1_Link2: origin xyz=0.19292766643937015 0 1 rpy=0 0 0 -> xyz=0.2962198806377458 0 1 rpy=0 0 0
- joint Link2_Link3: origin xyz=1.0713668230413884 0 0 rpy=0 0 0 -> xyz=0.5765937489915485 0 0 rpy=0 0 0
- joint Link3_Link4: origin xyz=1.0119438504694291 0 0 rpy=0 0 0 -> xyz=0.29048986510979236 0 0 rpy=0 0 0
- joint Link4_Link5: origin xyz=1.0688683422390406 0 0 rpy=0 0 0 -> xyz=0.6305169742925424 0 0 rpy=0 0 0
- joint Link5_Link6: origin xyz=0.5612359157856884 0 0 rpy=0 0 0 -> xyz=0.8361367164541827 0 0 rpy=0 0 0

File: body1.urdf (robot description, URDF)
Before this commit: robot robot, 9 links, 8 joints
Links:
- removed link Link8
- removed link Link9
- link Link1: geometry collision box size=0.4368359799180097 0.3742173587464101 0.5239036967877788; visual box size=0.4368359799180097 0.3742173587464101 0.5239036967877788
- link Link2: geometry collision box size=1.0379449590545313 0.8755786157589254 0.2292195779405017; visual box size=1.0379449590545313 0.8755786157589254 0.2292195779405017
- link Link3: geometry collision box size=0.6257496996613525 1.1747511208338357 0.6408398365171563; visual box size=0.6257496996613525 1.1747511208338357 0.6408398365171563
- link Link4: geometry collision box size=0.6382509851649013 1.0433666275402418 0.9104836932271464; visual box size=0.6382509851649013 1.0433666275402418 0.9104836932271464
- link Link5: geometry collision box size=0.7301553436685962 1.1241285409324717 0.971874775063979; visual box size=0.7301553436685962 1.1241285409324717 0.971874775063979
- link Link6: geometry collision box size=0.34071147991168405 1.2305882040305305 0.4753785133281391; visual box size=0.34071147991168405 1.2305882040305305 0.4753785133281391
- link Link7: geometry collision box size=0.5514294518802828 1.0031257337557253 0.4940543800621974; visual box size=0.5514294518802828 1.0031257337557253 0.4940543800621974
Joints:
- removed joint Link7_Link8
- removed joint Link8_Link9
- joint Link1_Link2: origin xyz=0.10210787919524374 0 1 rpy=0 0 0 -> xyz=0.21841798995900485 0 1 rpy=0 0 0
- joint Link2_Link3: origin xyz=0.5164588930811218 0 0 rpy=0 0 0 -> xyz=1.0379449590545313 0 0 rpy=0 0 0
- joint Link3_Link4: origin xyz=0.8833262706192718 0 0 rpy=0 0 0 -> xyz=0.6257496996613525 0 0 rpy=0 0 0
- joint Link4_Link5: origin xyz=0.3315467823120757 0 0 rpy=0 0 0 -> xyz=0.6382509851649013 0 0 rpy=0 0 0
- joint Link5_Link6: origin xyz=0.49402756202223086 0 0 rpy=0 0 0 -> xyz=0.7301553436685962 0 0 rpy=0 0 0
- joint Link6_Link7: origin xyz=0.8952719306418322 0 0 rpy=0 0 0 -> xyz=0.34071147991168405 0 0 rpy=0 0 0

File: body2.urdf (robot description, URDF)
Before this commit: robot robot, 12 links, 11 joints
Links:
- removed link Link11
- removed link Link12
- link Link1: geometry collision box size=0.30104922089568276 0.5017438094472846 0.4043317815649987; visual box size=0.30104922089568276 0.5017438094472846 0.4043317815649987
- link Link10: geometry collision box size=0.4899864929752684 0.7784408156118721 0.7529177529332011; visual box size=0.4899864929752684 0.7784408156118721 0.7529177529332011
- link Link2: geometry collision box size=0.13663314864488 1.2270051321432127 1.0492798634442857; visual box size=0.13663314864488 1.2270051321432127 1.0492798634442857
- link Link3: geometry collision box size=0.6756192946707114 0.7093773534254837 0.21040967881594383; visual box size=0.6756192946707114 0.7093773534254837 0.21040967881594383
- link Link4: geometry collision box size=0.2689888269216357 0.7858524727613225 1.128991845183794; visual box size=0.2689888269216357 0.7858524727613225 1.128991845183794
- link Link5: geometry collision box size=0.2335423985147226 1.2952056538714485 0.48748630829139916; visual box size=0.2335423985147226 1.2952056538714485 0.48748630829139916
- link Link6: geometry collision box size=0.1333995910443039 0.3500906414887112 0.8331720603773802; visual box size=0.1333995910443039 0.3500906414887112 0.8331720603773802
- link Link7: geometry collision box size=0.7950987422702129 1.0854225193494265 0.8783427597799949; visual box size=0.7950987422702129 1.0854225193494265 0.8783427597799949
- link Link8: geometry collision box size=0.7804696861867513 0.8383975601040179 0.15355577245916738; visual box size=0.7804696861867513 0.8383975601040179 0.15355577245916738
- link Link9: geometry collision box size=1.0659739827325314 0.34222261791158487 1.0867020645250731; visual box size=1.0659739827325314 0.34222261791158487 1.0867020645250731
Joints:
- removed joint Link10_Link11
- removed joint Link11_Link12
- joint Link1_Link2: origin xyz=0.40909000370546333 0 1 rpy=0 0 0 -> xyz=0.15052461044784138 0 1 rpy=0 0 0
- joint Link2_Link3: origin xyz=0.7923590534502866 0 0 rpy=0 0 0 -> xyz=0.13663314864488 0 0 rpy=0 0 0
- joint Link3_Link4: origin xyz=0.7533849456709687 0 0 rpy=0 0 0 -> xyz=0.6756192946707114 0 0 rpy=0 0 0
- joint Link4_Link5: origin xyz=0.3298802349316594 0 0 rpy=0 0 0 -> xyz=0.2689888269216357 0 0 rpy=0 0 0
- joint Link5_Link6: origin xyz=0.9075250993279642 0 0 rpy=0 0 0 -> xyz=0.2335423985147226 0 0 rpy=0 0 0
- joint Link6_Link7: origin xyz=0.9765111556423784 0 0 rpy=0 0 0 -> xyz=0.1333995910443039 0 0 rpy=0 0 0
- joint Link7_Link8: origin xyz=0.14228066732264935 0 0 rpy=0 0 0 -> xyz=0.7950987422702129 0 0 rpy=0 0 0
- joint Link8_Link9: origin xyz=0.5071773706300138 0 0 rpy=0 0 0 -> xyz=0.7804696861867513 0 0 rpy=0 0 0
- joint Link9_Link10: origin xyz=0.39029303910840696 0 0 rpy=0 0 0 -> xyz=1.0659739827325314 0 0 rpy=0 0 0

File: body3.urdf (robot description, URDF)
Before this commit: robot robot, 3 links, 2 joints
Links:
- added link Link10, mass 1; collision box size=0.19491509512090113 1.0108846685381407 0.585519298151279; visual box size=0.19491509512090113 1.0108846685381407 0.585519298151279
- added link Link4, mass 1; collision box size=0.17189115311860406 0.32757130329753575 0.21559238039442838; visual box size=0.17189115311860406 0.32757130329753575 0.21559238039442838
- added link Link5, mass 1; collision box size=0.9494234709093936 1.2437414870802257 0.7959999722705157; visual box size=0.9494234709093936 1.2437414870802257 0.7959999722705157
- added link Link6, mass 1; collision box size=0.8748032351243312 0.5746128079932047 0.953820008124712; visual box size=0.8748032351243312 0.5746128079932047 0.953820008124712
- added link Link7, mass 1; collision box size=0.7608973329846517 0.8166636300163108 0.3154399763586231; visual box size=0.7608973329846517 0.8166636300163108 0.3154399763586231
- added link Link8, mass 1; collision box size=0.45442336820441864 0.6122647708833411 0.6501923218249441; visual box size=0.45442336820441864 0.6122647708833411 0.6501923218249441
- added link Link9, mass 1; collision box size=0.7720167161660139 1.2897598273506279 0.5695980659440454; visual box size=0.7720167161660139 1.2897598273506279 0.5695980659440454
- link Link1: geometry collision box size=0.8303392835989039 0.7618293686097628 0.9885171816479413; visual box size=0.8303392835989039 0.7618293686097628 0.9885171816479413
- link Link2: geometry collision box size=0.9805869323470495 0.9134345879564159 0.753986032975756; visual box size=0.9805869323470495 0.9134345879564159 0.753986032975756
- link Link3: geometry collision box size=0.6265762595438173 0.8846401170046152 1.0885307974738747; visual box size=0.6265762595438173 0.8846401170046152 1.0885307974738747
Joints:
- added joint Link3_Link4: type revolute, parent Link3, child Link4, origin xyz=0.6265762595438173 0 0 rpy=0 0 0, axis 0 1 0, limit lower=-3.14159 upper=3.14159 effort=0.0 velocity=0.0
- added joint Link4_Link5: type revolute, parent Link4, child Link5, origin xyz=0.17189115311860406 0 0 rpy=0 0 0, axis 0 1 0, limit lower=-3.14159 upper=3.14159 effort=0.0 velocity=0.0
- added joint Link5_Link6: type revolute, parent Link5, child Link6, origin xyz=0.9494234709093936 0 0 rpy=0 0 0, axis 0 1 0, limit lower=-3.14159 upper=3.14159 effort=0.0 velocity=0.0
- added joint Link6_Link7: type revolute, parent Link6, child Link7, origin xyz=0.8748032351243312 0 0 rpy=0 0 0, axis 0 1 0, limit lower=-3.14159 upper=3.14159 effort=0.0 velocity=0.0
- added joint Link7_Link8: type revolute, parent Link7, child Link8, origin xyz=0.7608973329846517 0 0 rpy=0 0 0, axis 0 1 0, limit lower=-3.14159 upper=3.14159 effort=0.0 velocity=0.0
- added joint Link8_Link9: type revolute, parent Link8, child Link9, origin xyz=0.45442336820441864 0 0 rpy=0 0 0, axis 0 1 0, limit lower=-3.14159 upper=3.14159 effort=0.0 velocity=0.0
- added joint Link9_Link10: type revolute, parent Link9, child Link10, origin xyz=0.7720167161660139 0 0 rpy=0 0 0, axis 0 1 0, limit lower=-3.14159 upper=3.14159 effort=0.0 velocity=0.0
- joint Link1_Link2: origin xyz=0.5435234151950308 0 1 rpy=0 0 0 -> xyz=0.4151696417994519 0 1 rpy=0 0 0
- joint Link2_Link3: origin xyz=0.3715316684299145 0 0 rpy=0 0 0 -> xyz=0.9805869323470495 0 0 rpy=0 0 0

File: body4.urdf (robot description, URDF)
Before this commit: robot robot, 7 links, 6 joints
Links:
- link Link1: geometry collision box size=0.7951815254474893 1.125732064618343 0.37378760406311207; visual box size=0.7951815254474893 1.125732064618343 0.37378760406311207
- link Link2: geometry collision box size=0.484914315189496 1.1139037367702043 0.7000757915355218; visual box size=0.484914315189496 1.1139037367702043 0.7000757915355218
- link Link3: geometry collision box size=0.9568548998756946 0.5514789751606304 1.1330732627172408; visual box size=0.9568548998756946 0.5514789751606304 1.1330732627172408
- link Link4: geometry collision box size=0.9650490268235218 0.7809618422752105 0.25789709926481585; visual box size=0.9650490268235218 0.7809618422752105 0.25789709926481585
- link Link5: geometry collision box size=0.8091341598481231 0.9444627355497988 1.123339767688236; visual box size=0.8091341598481231 0.9444627355497988 1.123339767688236
- link Link6: geometry collision box size=0.15335345671953063 0.9981849336486841 0.9584468357271864; visual box size=0.15335345671953063 0.9981849336486841 0.9584468357271864
- link Link7: geometry collision box size=1.0043735899815993 0.6524601733936395 0.8427098058791798; visual box size=1.0043735899815993 0.6524601733936395 0.8427098058791798
Joints:
- joint Link1_Link2: origin xyz=0.17151808149661996 0 1 rpy=0 0 0 -> xyz=0.39759076272374466 0 1 rpy=0 0 0
- joint Link2_Link3: origin xyz=0.8380803891788293 0 0 rpy=0 0 0 -> xyz=0.484914315189496 0 0 rpy=0 0 0
- joint Link3_Link4: origin xyz=0.238653574247247 0 0 rpy=0 0 0 -> xyz=0.9568548998756946 0 0 rpy=0 0 0
- joint Link4_Link5: origin xyz=0.8496985649243783 0 0 rpy=0 0 0 -> xyz=0.9650490268235218 0 0 rpy=0 0 0
- joint Link5_Link6: origin xyz=0.39031000932257554 0 0 rpy=0 0 0 -> xyz=0.8091341598481231 0 0 rpy=0 0 0
- joint Link6_Link7: origin xyz=0.357688454730666 0 0 rpy=0 0 0 -> xyz=0.15335345671953063 0 0 rpy=0 0 0
