Commit message: 1dmorph done

File: body0.urdf (robot description, URDF)
Before this commit: robot robot, 6 links, 5 joints
Links:
- added link Link10, mass 1; collision box size=1.0082202561230638 1.2362700946211012 0.8755549385891939; visual box size=1.0082202561230638 1.2362700946211012 0.8755549385891939
- added link Link11, mass 1; collision box size=0.3186170179565718 0.5160210182126961 0.7912040640923101; visual box size=0.3186170179565718 0.5160210182126961 0.7912040640923101
- added link Link7, mass 1; collision box size=0.3381177987744107 0.6199002911310034 0.5038335501925308; visual box size=0.3381177987744107 0.6199002911310034 0.5038335501925308
- added link Link8, mass 1; collision box size=0.22151159953498414 0.3819270412931542 0.2112576752647539; visual box size=0.22151159953498414 0.3819270412931542 0.2112576752647539
- added link Link9, mass 1; collision box size=0.4845058558251242 1.1879709544491648 0.6454173093999709; visual box size=0.4845058558251242 1.1879709544491648 0.6454173093999709
- link Link1: geometry collision box size=0.8062232683847931 0.9665153036640386 0.7318631557242138; visual box size=0.8062232683847931 0.9665153036640386 0.7318631557242138
- link Link2: geometry collision box size=0.29989982358157485 1.0981641928021637 0.9095517071351987; visual box size=0.29989982358157485 1.0981641928021637 0.9095517071351987
- link Link3: geometry collision box size=1.0782101016901844 1.284197994774307 1.059407734644185; visual box size=1.0782101016901844 1.284197994774307 1.059407734644185
- link Link4: geometry collision box size=0.5231109203084756 0.6352642583398438 0.8983164858620981; visual box size=0.5231109203084756 0.6352642583398438 0.8983164858620981
- link Link5: geometry collision box size=0.7165974767603834 1.0943671413096685 0.7704951111184082; visual box size=0.7165974767603834 1.0943671413096685 0.7704951111184082
- link Link6: geometry collision box size=0.8355680060377663 0.417952984135382 1.0147316617255986; visual box size=0.8355680060377663 0.417952984135382 1.0147316617255986
Joints:
- added joint Link10_Link11: type revolute, parent Link10, child Link11, origin xyz=1.0082202561230638 0 0 rpy=0 0 0, axis 0 1 0, limit lower=-3.14159 upper=3.14159 effort=0.0 velocity=0.0
- added joint Link6_Link7: type revolute, parent Link6, child Link7, origin xyz=0.8355680060377663 0 0 rpy=0 0 0, axis 0 1 0, limit lower=-3.14159 upper=3.14159 effort=0.0 velocity=0.0
- added joint Link7_Link8: type revolute, parent Link7, child Link8, origin xyz=0.3381177987744107 0 0 rpy=0 0 0, axis 0 1 0, limit lower=-3.14159 upper=3.14159 effort=0.0 velocity=0.0
- added joint Link8_Link9: type revolute, parent Link8, child Link9, origin xyz=0.22151159953498414 0 0 rpy=0 0 0, axis 0 1 0, limit lower=-3.14159 upper=3.14159 effort=0.0 velocity=0.0
- added joint Link9_Link10: type revolute, parent Link9, child Link10, origin xyz=0.4845058558251242 0 0 rpy=0 0 0, axis 0 1 0, limit lower=-3.14159 upper=3.14159 effort=0.0 velocity=0.0
- joint Link1_Link2: origin xyz=0.2962198806377458 0 1 rpy=0 0 0 -> xyz=0.40311163419239654 0 1 rpy=0 0 0
- joint Link2_Link3: origin xyz=0.5765937489915485 0 0 rpy=0 0 0 -> xyz=0.29989982358157485 0 0 rpy=0 0 0
- joint Link3_Link4: origin xyz=0.29048986510979236 0 0 rpy=0 0 0 -> xyz=1.0782101016901844 0 0 rpy=0 0 0
- joint Link4_Link5: origin xyz=0.6305169742925424 0 0 rpy=0 0 0 -> xyz=0.5231109203084756 0 0 rpy=0 0 0
- joint Link5_Link6: origin xyz=0.8361367164541827 0 0 rpy=0 0 0 -> xyz=0.7165974767603834 0 0 rpy=0 0 0

File: body1.urdf (robot description, URDF)
Before this commit: robot robot, 7 links, 6 joints
Links:
- added link Link10, mass 1; collision box size=0.8630886585298222 0.6179384118152544 0.4692631792495394; visual box size=0.8630886585298222 0.6179384118152544 0.4692631792495394
- added link Link8, mass 1; collision box size=0.9638447846674751 1.2148373316877432 0.21799288852548956; visual box size=0.9638447846674751 1.2148373316877432 0.21799288852548956
- added link Link9, mass 1; collision box size=0.38835478852657335 1.1022046944064818 1.038790228608312; visual box size=0.38835478852657335 1.1022046944064818 1.038790228608312
- link Link1: geometry collision box size=0.34571478631004815 1.0193309140689324 0.4454742653874615; visual box size=0.34571478631004815 1.0193309140689324 0.4454742653874615
- link Link2: geometry collision box size=0.7209191233098056 0.4586417034089741 1.1266634049570077; visual box size=0.7209191233098056 0.4586417034089741 1.1266634049570077
- link Link3: geometry collision box size=1.065066722947524 0.4169615662571639 0.28156375236143794; visual box size=1.065066722947524 0.4169615662571639 0.28156375236143794
- link Link4: geometry collision box size=0.561609928819149 0.516590110102868 0.652441254627209; visual box size=0.561609928819149 0.516590110102868 0.652441254627209
- link Link5: geometry collision box size=0.8486952110104009 0.3431633167374623 0.3409242486892765; visual box size=0.8486952110104009 0.3431633167374623 0.3409242486892765
- link Link6: geometry collision box size=0.4707464621980194 0.47568840376256266 0.21616765033126903; visual box size=0.4707464621980194 0.47568840376256266 0.21616765033126903
- link Link7: geometry collision box size=0.6982756471783486 0.8013559890561399 0.7924836993592211; visual box size=0.6982756471783486 0.8013559890561399 0.7924836993592211
Joints:
- added joint Link7_Link8: type revolute, parent Link7, child Link8, origin xyz=0.6982756471783486 0 0 rpy=0 0 0, axis 0 1 0, limit lower=-3.14159 upper=3.14159 effort=0.0 velocity=0.0
- added joint Link8_Link9: type revolute, parent Link8, child Link9, origin xyz=0.9638447846674751 0 0 rpy=0 0 0, axis 0 1 0, limit lower=-3.14159 upper=3.14159 effort=0.0 velocity=0.0
- added joint Link9_Link10: type revolute, parent Link9, child Link10, origin xyz=0.38835478852657335 0 0 rpy=0 0 0, axis 0 1 0, limit lower=-3.14159 upper=3.14159 effort=0.0 velocity=0.0
- joint Link1_Link2: origin xyz=0.21841798995900485 0 1 rpy=0 0 0 -> xyz=0.17285739315502407 0 1 rpy=0 0 0
- joint Link2_Link3: origin xyz=1.0379449590545313 0 0 rpy=0 0 0 -> xyz=0.7209191233098056 0 0 rpy=0 0 0
- joint Link3_Link4: origin xyz=0.6257496996613525 0 0 rpy=0 0 0 -> xyz=1.065066722947524 0 0 rpy=0 0 0
- joint Link4_Link5: origin xyz=0.6382509851649013 0 0 rpy=0 0 0 -> xyz=0.561609928819149 0 0 rpy=0 0 0
- joint Link5_Link6: origin xyz=0.7301553436685962 0 0 rpy=0 0 0 -> xyz=0.8486952110104009 0 0 rpy=0 0 0
- joint Link6_Link7: origin xyz=0.34071147991168405 0 0 rpy=0 0 0 -> xyz=0.4707464621980194 0 0 rpy=0 0 0

File: body2.urdf (robot description, URDF)
Before this commit: robot robot, 10 links, 9 joints
Links:
- added link Link11, mass 1; collision box size=0.45417345338506176 1.110995171033885 0.5591242123943702; visual box size=0.45417345338506176 1.110995171033885 0.5591242123943702
- link Link1: geometry collision box size=0.9595251606306096 1.061350361371912 1.0839613320442556; visual box size=0.9595251606306096 1.061350361371912 1.0839613320442556
- link Link10: geometry collision box size=0.4116767708280027 0.4840915069330652 0.5146078305621253; visual box size=0.4116767708280027 0.4840915069330652 0.5146078305621253
- link Link2: geometry collision box size=0.9647207843447262 0.3077258600972304 0.7841477772356458; visual box size=0.9647207843447262 0.3077258600972304 0.7841477772356458
- link Link3: geometry collision box size=0.23511216607937338 0.6517870820566625 0.9969199251607769; visual box size=0.23511216607937338 0.6517870820566625 0.9969199251607769
- link Link4: geometry collision box size=0.17517868942662032 1.0568055461718653 0.683653722901709; visual box size=0.17517868942662032 1.0568055461718653 0.683653722901709
- link Link5: geometry collision box size=0.3232523383104292 0.4801936977685681 0.20627140337105063; visual box size=0.3232523383104292 0.4801936977685681 0.20627140337105063
- link Link6: geometry collision box size=1.0964325180771952 0.8553717801163367 0.6507758442195755; visual box size=1.0964325180771952 0.8553717801163367 0.6507758442195755
- link Link7: geometry collision box size=0.5908124752429524 0.43239837564249445 0.35948189096797045; visual box size=0.5908124752429524 0.43239837564249445 0.35948189096797045
- link Link8: geometry collision box size=0.7865184134964147 1.2948417679318043 0.6446652611264142; visual box size=0.7865184134964147 1.2948417679318043 0.6446652611264142
- link Link9: geometry collision box size=0.26634875291404747 0.37805320059117403 0.897420744343846; visual box size=0.26634875291404747 0.37805320059117403 0.897420744343846
Joints:
- added joint Link10_Link11: type revolute, parent Link10, child Link11, origin xyz=0.4116767708280027 0 0 rpy=0 0 0, axis 0 1 0, limit lower=-3.14159 upper=3.14159 effort=0.0 velocity=0.0
- joint Link1_Link2: origin xyz=0.15052461044784138 0 1 rpy=0 0 0 -> xyz=0.4797625803153048 0 1 rpy=0 0 0
- joint Link2_Link3: origin xyz=0.13663314864488 0 0 rpy=0 0 0 -> xyz=0.9647207843447262 0 0 rpy=0 0 0
- joint Link3_Link4: origin xyz=0.6756192946707114 0 0 rpy=0 0 0 -> xyz=0.23511216607937338 0 0 rpy=0 0 0
- joint Link4_Link5: origin xyz=0.2689888269216357 0 0 rpy=0 0 0 -> xyz=0.17517868942662032 0 0 rpy=0 0 0
- joint Link5_Link6: origin xyz=0.2335423985147226 0 0 rpy=0 0 0 -> xyz=0.3232523383104292 0 0 rpy=0 0 0
- joint Link6_Link7: origin xyz=0.1333995910443039 0 0 rpy=0 0 0 -> xyz=1.0964325180771952 0 0 rpy=0 0 0
- joint Link7_Link8: origin xyz=0.7950987422702129 0 0 rpy=0 0 0 -> xyz=0.5908124752429524 0 0 rpy=0 0 0
- joint Link8_Link9: origin xyz=0.7804696861867513 0 0 rpy=0 0 0 -> xyz=0.7865184134964147 0 0 rpy=0 0 0
- joint Link9_Link10: origin xyz=1.0659739827325314 0 0 rpy=0 0 0 -> xyz=0.26634875291404747 0 0 rpy=0 0 0

File: body3.urdf (robot description, URDF)
Before this commit: robot robot, 10 links, 9 joints
Links:
- added link Link11, mass 1; collision box size=0.327176537865173 0.8927557858529982 0.29153499276129935; visual box size=0.327176537865173 0.8927557858529982 0.29153499276129935
- added link Link12, mass 1; collision box size=0.9048371763706426 1.2204779810796984 1.1397980507938994; visual box size=0.9048371763706426 1.2204779810796984 1.1397980507938994
- link Link1: geometry collision box size=0.45857056444092936 1.1940512610773886 0.6514965495005806; visual box size=0.45857056444092936 1.1940512610773886 0.6514965495005806
- link Link10: geometry collision box size=0.753935019927969 0.6974531898693352 1.1423229917813211; visual box size=0.753935019927969 0.6974531898693352 1.1423229917813211
- link Link2: geometry collision box size=0.6491329872787547 0.8024864722532397 0.837417122641938; visual box size=0.6491329872787547 0.8024864722532397 0.837417122641938
- link Link3: geometry collision box size=0.44408759745345716 1.0944185341768846 1.0015539419595552; visual box size=0.44408759745345716 1.0944185341768846 1.0015539419595552
- link Link4: geometry collision box size=0.2432031018558455 0.4748632461722811 0.7204521464283461; visual box size=0.2432031018558455 0.4748632461722811 0.7204521464283461
- link Link5: geometry collision box size=0.7119836079215836 1.0672890717397463 0.5782033005109191; visual box size=0.7119836079215836 1.0672890717397463 0.5782033005109191
- link Link6: geometry collision box size=0.13713335844305877 0.8990550273423357 0.9194563342008288; visual box size=0.13713335844305877 0.8990550273423357 0.9194563342008288
- link Link7: geometry collision box size=0.5241193156010672 0.32207426654827914 0.9117230991681002; visual box size=0.5241193156010672 0.32207426654827914 0.9117230991681002
- link Link8: geometry collision box size=0.19165834341197976 0.6814811372087779 0.21204248135049106; visual box size=0.19165834341197976 0.6814811372087779 0.21204248135049106
- link Link9: geometry collision box size=0.49243885640763674 0.8335248273433946 0.4121681953151539; visual box size=0.49243885640763674 0.8335248273433946 0.4121681953151539
Joints:
- added joint Link10_Link11: type revolute, parent Link10, child Link11, origin xyz=0.753935019927969 0 0 rpy=0 0 0, axis 0 1 0, limit lower=-3.14159 upper=3.14159 effort=0.0 velocity=0.0
- added joint Link11_Link12: type revolute, parent Link11, child Link12, origin xyz=0.327176537865173 0 0 rpy=0 0 0, axis 0 1 0, limit lower=-3.14159 upper=3.14159 effort=0.0 velocity=0.0
- joint Link1_Link2: origin xyz=0.4151696417994519 0 1 rpy=0 0 0 -> xyz=0.22928528222046468 0 1 rpy=0 0 0
- joint Link2_Link3: origin xyz=0.9805869323470495 0 0 rpy=0 0 0 -> xyz=0.6491329872787547 0 0 rpy=0 0 0
- joint Link3_Link4: origin xyz=0.6265762595438173 0 0 rpy=0 0 0 -> xyz=0.44408759745345716 0 0 rpy=0 0 0
- joint Link4_Link5: origin xyz=0.17189115311860406 0 0 rpy=0 0 0 -> xyz=0.2432031018558455 0 0 rpy=0 0 0
- joint Link5_Link6: origin xyz=0.9494234709093936 0 0 rpy=0 0 0 -> xyz=0.7119836079215836 0 0 rpy=0 0 0
- joint Link6_Link7: origin xyz=0.8748032351243312 0 0 rpy=0 0 0 -> xyz=0.13713335844305877 0 0 rpy=0 0 0
- joint Link7_Link8: origin xyz=0.7608973329846517 0 0 rpy=0 0 0 -> xyz=0.5241193156010672 0 0 rpy=0 0 0
- joint Link8_Link9: origin xyz=0.45442336820441864 0 0 rpy=0 0 0 -> xyz=0.19165834341197976 0 0 rpy=0 0 0
- joint Link9_Link10: origin xyz=0.7720167161660139 0 0 rpy=0 0 0 -> xyz=0.49243885640763674 0 0 rpy=0 0 0

File: body4.urdf (robot description, URDF)
Before this commit: robot robot, 7 links, 6 joints
Links:
- added link Link8, mass 1; collision box size=0.9864571033716669 0.644399499812023 0.3529407433061834; visual box size=0.9864571033716669 0.644399499812023 0.3529407433061834
- added link Link9, mass 1; collision box size=0.40399793975566267 1.176840005012554 0.31669929482183845; visual box size=0.40399793975566267 1.176840005012554 0.31669929482183845
- link Link1: geometry collision box size=0.5878955716500622 0.623547084403604 0.43168663693708587; visual box size=0.5878955716500622 0.623547084403604 0.43168663693708587
- link Link2: geometry collision box size=0.21743783216509274 0.39396668233577287 1.0070234572876111; visual box size=0.21743783216509274 0.39396668233577287 1.0070234572876111
- link Link3: geometry collision box size=0.20793277546638214 0.40547243639530056 0.9977278806522789; visual box size=0.20793277546638214 0.40547243639530056 0.9977278806522789
- link Link4: geometry collision box size=0.3392779693334449 0.8538763170771249 0.8508833520835417; visual box size=0.3392779693334449 0.8538763170771249 0.8508833520835417
- link Link5: geometry collision box size=0.7682240711212576 1.0000883812602666 0.1898776085079051; visual box size=0.7682240711212576 1.0000883812602666 0.1898776085079051
- link Link6: geometry collision box size=0.3174534988171348 0.5493629727727474 0.5948643062450626; visual box size=0.3174534988171348 0.5493629727727474 0.5948643062450626
- link Link7: geometry collision box size=0.3296170688120803 1.0866062588405283 0.8594996685312948; visual box size=0.3296170688120803 1.0866062588405283 0.8594996685312948
Joints:
- added joint Link7_Link8: type revolute, parent Link7, child Link8, origin xyz=0.3296170688120803 0 0 rpy=0 0 0, axis 0 1 0, limit lower=-3.14159 upper=3.14159 effort=0.0 velocity=0.0
- added joint Link8_Link9: type revolute, parent Link8, child Link9, origin xyz=0.9864571033716669 0 0 rpy=0 0 0, axis 0 1 0, limit lower=-3.14159 upper=3.14159 effort=0.0 velocity=0.0
- joint Link1_Link2: origin xyz=0.39759076272374466 0 1 rpy=0 0 0 -> xyz=0.2939477858250311 0 1 rpy=0 0 0
- joint Link2_Link3: origin xyz=0.484914315189496 0 0 rpy=0 0 0 -> xyz=0.21743783216509274 0 0 rpy=0 0 0
- joint Link3_Link4: origin xyz=0.9568548998756946 0 0 rpy=0 0 0 -> xyz=0.20793277546638214 0 0 rpy=0 0 0
- joint Link4_Link5: origin xyz=0.9650490268235218 0 0 rpy=0 0 0 -> xyz=0.3392779693334449 0 0 rpy=0 0 0
- joint Link5_Link6: origin xyz=0.8091341598481231 0 0 rpy=0 0 0 -> xyz=0.7682240711212576 0 0 rpy=0 0 0
- joint Link6_Link7: origin xyz=0.15335345671953063 0 0 rpy=0 0 0 -> xyz=0.3174534988171348 0 0 rpy=0 0 0

Commit message: map generating properly

File: body0.urdf (robot description, URDF)
Before this commit: robot robot, 11 links, 10 joints
Links:
- removed link Link10
- removed link Link11
- removed link Link9
- link Link1: geometry collision box size=0.18524316791383846 0.7567274918080313 0.31922015871615816; visual box size=0.18524316791383846 0.7567274918080313 0.31922015871615816
- link Link2: geometry collision box size=0.2905833444310285 0.8586903293803039 1.1278093853114792; visual box size=0.2905833444310285 0.8586903293803039 1.1278093853114792
- link Link3: geometry collision box size=0.39762768816159455 0.7978013244484499 0.5290514661207105; visual box size=0.39762768816159455 0.7978013244484499 0.5290514661207105
- link Link4: geometry collision box size=0.7131530373772446 0.565641174934226 0.9018228054755174; visual box size=0.7131530373772446 0.565641174934226 0.9018228054755174
- link Link5: geometry collision box size=0.1939154646345829 0.9212797462297067 0.2031175899548466; visual box size=0.1939154646345829 0.9212797462297067 0.2031175899548466
- link Link6: geometry collision box size=0.7074454575731063 0.5257673226977451 0.9238783822360239; visual box size=0.7074454575731063 0.5257673226977451 0.9238783822360239
- link Link7: geometry collision box size=0.8626519384727511 0.8268794095679535 0.7631641300245005; visual box size=0.8626519384727511 0.8268794095679535 0.7631641300245005
- link Link8: geometry collision box size=0.8701387850586967 0.6854528086314946 0.6748060565751169; visual box size=0.8701387850586967 0.6854528086314946 0.6748060565751169
Joints:
- removed joint Link10_Link11
- removed joint Link8_Link9
- removed joint Link9_Link10
- joint Link1_Link2: origin xyz=0.40311163419239654 0 1 rpy=0 0 0 -> xyz=0.09262158395691923 0 1 rpy=0 0 0
- joint Link2_Link3: origin xyz=0.29989982358157485 0 0 rpy=0 0 0 -> xyz=0.2905833444310285 0 0 rpy=0 0 0
- joint Link3_Link4: origin xyz=1.0782101016901844 0 0 rpy=0 0 0 -> xyz=0.39762768816159455 0 0 rpy=0 0 0
- joint Link4_Link5: origin xyz=0.5231109203084756 0 0 rpy=0 0 0 -> xyz=0.7131530373772446 0 0 rpy=0 0 0
- joint Link5_Link6: origin xyz=0.7165974767603834 0 0 rpy=0 0 0 -> xyz=0.1939154646345829 0 0 rpy=0 0 0
- joint Link6_Link7: origin xyz=0.8355680060377663 0 0 rpy=0 0 0 -> xyz=0.7074454575731063 0 0 rpy=0 0 0
- joint Link7_Link8: origin xyz=0.3381177987744107 0 0 rpy=0 0 0 -> xyz=0.8626519384727511 0 0 rpy=0 0 0

Commit message: done with 3d-morph map!!!

File: body0.urdf (robot description, URDF)
Before this commit: robot robot, 8 links, 7 joints
Links:
- removed link Link5
- removed link Link6
- removed link Link7
- removed link Link8
- added link Link0, mass 1; collision box size=1 1 1; visual box size=1 1 1
- link Link1: geometry collision box size=1 1 1; visual box size=1 1 1
- link Link2: geometry collision box size=1 1 1; visual box size=1 1 1
- link Link3: geometry collision box size=1 1 1; visual box size=1 1 1
- link Link4: geometry collision box size=1 1 1; visual box size=1 1 1
Joints:
- removed joint Link4_Link5
- removed joint Link5_Link6
- removed joint Link6_Link7
- removed joint Link7_Link8
- added joint Link0_Link1: type revolute, parent Link0, child Link1, origin xyz=-0.5 0.0 1.0 rpy=0 0 0, axis 0 1 0, limit lower=-3.14159 upper=3.14159 effort=0.0 velocity=0.0
- joint Link1_Link2: axis 0 1 0 -> 0 0 1; origin xyz=0.09262158395691923 0 1 rpy=0 0 0 -> xyz=-0.5 0.0 0.5 rpy=0 0 0
- joint Link2_Link3: axis 0 1 0 -> 1 0 0; origin xyz=0.2905833444310285 0 0 rpy=0 0 0 -> xyz=0.0 -0.5 0.5 rpy=0 0 0
- joint Link3_Link4: axis 0 1 0 -> 1 0 0; origin xyz=0.39762768816159455 0 0 rpy=0 0 0 -> xyz=0 -1 0 rpy=0 0 0
