Commit message: random bot evolution, submitted

File: body0.urdf (robot description, URDF)
Before this commit: robot robot, 7 links, 6 joints
Links:
- added link Link10, mass 1; collision box size=1 1 1; visual box size=1 1 1
- added link Link11, mass 1; collision box size=1 1 1; visual box size=1 1 1
- added link Link7, mass 1; collision box size=1 1 1; visual box size=1 1 1
- added link Link8, mass 1; collision box size=1 1 1; visual box size=1 1 1
- added link Link9, mass 1; collision box size=1 1 1; visual box size=1 1 1
Joints:
- removed joint Link0_Link5
- removed joint Link1_Link3
- removed joint Link1_Link6
- added joint Link1_Link5: type revolute, parent Link1, child Link5, origin xyz=0 1 0 rpy=0 0 0, axis 1 0 0, limit lower=-3.14159 upper=3.14159 effort=0.0 velocity=0.0
- added joint Link2_Link3: type revolute, parent Link2, child Link3, origin xyz=-0.5 0.0 0.5 rpy=0 0 0, axis 0 1 0, limit lower=-3.14159 upper=3.14159 effort=0.0 velocity=0.0
- added joint Link3_Link6: type revolute, parent Link3, child Link6, origin xyz=-0.5 -0.5 0.0 rpy=0 0 0, axis 1 0 0, limit lower=-3.14159 upper=3.14159 effort=0.0 velocity=0.0
- added joint Link3_Link7: type revolute, parent Link3, child Link7, origin xyz=-0.5 0.5 0.0 rpy=0 0 0, axis 1 0 0, limit lower=-3.14159 upper=3.14159 effort=0.0 velocity=0.0
- added joint Link5_Link8: type revolute, parent Link5, child Link8, origin xyz=0 1 0 rpy=0 0 0, axis 1 0 0, limit lower=-3.14159 upper=3.14159 effort=0.0 velocity=0.0
- added joint Link6_Link9: type revolute, parent Link6, child Link9, origin xyz=0 -1 0 rpy=0 0 0, axis 1 0 0, limit lower=-3.14159 upper=3.14159 effort=0.0 velocity=0.0
- added joint Link8_Link10: type revolute, parent Link8, child Link10, origin xyz=0 1 0 rpy=0 0 0, axis 1 0 0, limit lower=-3.14159 upper=3.14159 effort=0.0 velocity=0.0
- added joint Link9_Link11: type revolute, parent Link9, child Link11, origin xyz=0.5 -0.5 0.0 rpy=0 0 0, axis 0 1 0, limit lower=-3.14159 upper=3.14159 effort=0.0 velocity=0.0
- joint Link0_Link1: origin xyz=0.0 -0.5 1.0 rpy=0 0 0 -> xyz=0.0 0.5 1.0 rpy=0 0 0
- joint Link1_Link2: axis 0 1 0 -> 0 0 1; origin xyz=0.5 -0.5 0.0 rpy=0 0 0 -> xyz=0.0 0.5 0.5 rpy=0 0 0
- joint Link2_Link4: origin xyz=0.5 0.5 0.0 rpy=0 0 0 -> xyz=0.0 -0.5 0.5 rpy=0 0 0

File: body1.urdf (robot description, URDF)
Before this commit: robot robot, 6 links, 5 joints
Links:
- added link Link6, mass 1; collision box size=1 1 1; visual box size=1 1 1
- added link Link7, mass 1; collision box size=1 1 1; visual box size=1 1 1
Joints:
- removed joint Link0_Link5
- added joint Link0_Link6: type revolute, parent Link0, child Link6, origin xyz=-0.5 0.0 1.0 rpy=0 0 0, axis 0 1 0, limit lower=-3.14159 upper=3.14159 effort=0.0 velocity=0.0
- added joint Link2_Link7: type revolute, parent Link2, child Link7, origin xyz=-0.5 0.0 0.5 rpy=0 0 0, axis 0 1 0, limit lower=-3.14159 upper=3.14159 effort=0.0 velocity=0.0
- added joint Link4_Link5: type revolute, parent Link4, child Link5, origin xyz=0.5 -0.5 0.0 rpy=0 0 0, axis 1 0 0, limit lower=-3.14159 upper=3.14159 effort=0.0 velocity=0.0
- joint Link0_Link1: origin xyz=0.0 -0.5 1.0 rpy=0 0 0 -> xyz=0.0 0.5 1.0 rpy=0 0 0
- joint Link1_Link2: axis 1 0 0 -> 0 0 1; origin xyz=0 -1 0 rpy=0 0 0 -> xyz=0.0 0.5 0.5 rpy=0 0 0
- joint Link1_Link4: origin xyz=-0.5 -0.5 0.0 rpy=0 0 0 -> xyz=0.5 0.5 0.0 rpy=0 0 0

File: body2.urdf (robot description, URDF)
Before this commit: robot robot, 8 links, 7 joints
Links:
- added link Link10, mass 1; collision box size=1 1 1; visual box size=1 1 1
- added link Link11, mass 1; collision box size=1 1 1; visual box size=1 1 1
- added link Link8, mass 1; collision box size=1 1 1; visual box size=1 1 1
- added link Link9, mass 1; collision box size=1 1 1; visual box size=1 1 1
Joints:
- removed joint Link0_Link2
- removed joint Link2_Link5
- removed joint Link2_Link7
- removed joint Link3_Link4
- removed joint Link3_Link6
- added joint Link0_Link5: type revolute, parent Link0, child Link5, origin xyz=-0.5 0.0 1.0 rpy=0 0 0, axis 0 1 0, limit lower=-3.14159 upper=3.14159 effort=0.0 velocity=0.0
- added joint Link0_Link8: type revolute, parent Link0, child Link8, origin xyz=0.0 0.5 1.0 rpy=0 0 0, axis 1 0 0, limit lower=-3.14159 upper=3.14159 effort=0.0 velocity=0.0
- added joint Link1_Link2: type revolute, parent Link1, child Link2, origin xyz=0 -1 0 rpy=0 0 0, axis 1 0 0, limit lower=-3.14159 upper=3.14159 effort=0.0 velocity=0.0
- added joint Link1_Link4: type revolute, parent Link1, child Link4, origin xyz=0.5 -0.5 0.0 rpy=0 0 0, axis 0 1 0, limit lower=-3.14159 upper=3.14159 effort=0.0 velocity=0.0
- added joint Link1_Link6: type revolute, parent Link1, child Link6, origin xyz=0.0 -0.5 0.5 rpy=0 0 0, axis 0 0 1, limit lower=-3.14159 upper=3.14159 effort=0.0 velocity=0.0
- added joint Link3_Link11: type revolute, parent Link3, child Link11, origin xyz=0.0 -0.5 0.5 rpy=0 0 0, axis 0 0 1, limit lower=-3.14159 upper=3.14159 effort=0.0 velocity=0.0
- added joint Link4_Link9: type revolute, parent Link4, child Link9, origin xyz=0.5 -0.5 0.0 rpy=0 0 0, axis 1 0 0, limit lower=-3.14159 upper=3.14159 effort=0.0 velocity=0.0
- added joint Link5_Link7: type revolute, parent Link5, child Link7, origin xyz=-0.5 -0.5 0.0 rpy=0 0 0, axis 1 0 0, limit lower=-3.14159 upper=3.14159 effort=0.0 velocity=0.0
- added joint Link8_Link10: type revolute, parent Link8, child Link10, origin xyz=-0.5 0.5 0.0 rpy=0 0 0, axis 0 1 0, limit lower=-3.14159 upper=3.14159 effort=0.0 velocity=0.0
- joint Link0_Link1: axis 0 1 0 -> 1 0 0; origin xyz=-0.5 0.0 1.0 rpy=0 0 0 -> xyz=0.0 -0.5 1.0 rpy=0 0 0
- joint Link2_Link3: origin xyz=0 1 0 rpy=0 0 0 -> xyz=0 -1 0 rpy=0 0 0

File: body3.urdf (robot description, URDF)
Before this commit: robot robot, 9 links, 8 joints
Links:
- removed link Link8
- removed link Link9
- added link Link7, mass 1; collision box size=1 1 1; visual box size=1 1 1
Joints:
- removed joint Link0_Link3
- removed joint Link0_Link5
- removed joint Link0_Link8
- removed joint Link1_Link2
- removed joint Link5_Link6
- removed joint Link6_Link9
- added joint Link0_Link2: type revolute, parent Link0, child Link2, origin xyz=0.0 0.5 1.0 rpy=0 0 0, axis 1 0 0, limit lower=-3.14159 upper=3.14159 effort=0.0 velocity=0.0
- added joint Link0_Link6: type revolute, parent Link0, child Link6, origin xyz=0.5 0.0 1.0 rpy=0 0 0, axis 0 1 0, limit lower=-3.14159 upper=3.14159 effort=0.0 velocity=0.0
- added joint Link1_Link3: type revolute, parent Link1, child Link3, origin xyz=0.0 -0.5 0.5 rpy=0 0 0, axis 0 0 1, limit lower=-3.14159 upper=3.14159 effort=0.0 velocity=0.0
- added joint Link3_Link5: type revolute, parent Link3, child Link5, origin xyz=-0.5 0.0 0.5 rpy=0 0 0, axis 0 1 0, limit lower=-3.14159 upper=3.14159 effort=0.0 velocity=0.0
- added joint Link5_Link7: type revolute, parent Link5, child Link7, origin xyz=-1 0 0 rpy=0 0 0, axis 0 1 0, limit lower=-3.14159 upper=3.14159 effort=0.0 velocity=0.0
- joint Link0_Link1: axis 0 1 0 -> 1 0 0; origin xyz=-0.5 0.0 1.0 rpy=0 0 0 -> xyz=0.0 -0.5 1.0 rpy=0 0 0
- joint Link3_Link4: origin xyz=0 -1 0 rpy=0 0 0 -> xyz=0.0 -0.5 0.5 rpy=0 0 0

File: body4.urdf (robot description, URDF)
Before this commit: robot robot, 10 links, 9 joints
Links:
- removed link Link8
- removed link Link9
Joints:
- removed joint Link0_Link9
- removed joint Link1_Link4
- removed joint Link2_Link3
- removed joint Link4_Link8
- removed joint Link5_Link6
- removed joint Link5_Link7
- added joint Link0_Link3: type revolute, parent Link0, child Link3, origin xyz=0.5 0.0 1.0 rpy=0 0 0, axis 0 1 0, limit lower=-3.14159 upper=3.14159 effort=0.0 velocity=0.0
- added joint Link0_Link6: type revolute, parent Link0, child Link6, origin xyz=-0.5 0.0 1.0 rpy=0 0 0, axis 0 1 0, limit lower=-3.14159 upper=3.14159 effort=0.0 velocity=0.0
- added joint Link3_Link4: type revolute, parent Link3, child Link4, origin xyz=0.5 0.5 0.0 rpy=0 0 0, axis 1 0 0, limit lower=-3.14159 upper=3.14159 effort=0.0 velocity=0.0
- added joint Link4_Link7: type revolute, parent Link4, child Link7, origin xyz=0.0 0.5 0.5 rpy=0 0 0, axis 0 0 1, limit lower=-3.14159 upper=3.14159 effort=0.0 velocity=0.0
- joint Link0_Link1: axis 0 0 1 -> 1 0 0; origin xyz=0.0 0.0 1.5 rpy=0 0 0 -> xyz=0.0 0.5 1.0 rpy=0 0 0
- joint Link4_Link5: axis 0 1 0 -> 1 0 0; origin xyz=-0.5 0.5 0.0 rpy=0 0 0 -> xyz=0 1 0 rpy=0 0 0
