Commit message: done with code

File: body0.urdf (robot description, URDF)
Before this commit: robot robot, 13 links, 12 joints
Links:
- removed link Link10
- removed link Link11
- removed link Link12
- removed link Link9
Joints:
- removed joint Link0_Link3
- removed joint Link1_Link6
- removed joint Link2_Link4
- removed joint Link3_Link7
- removed joint Link4_Link9
- removed joint Link5_Link8
- removed joint Link6_Link10
- removed joint Link7_Link11
- removed joint Link7_Link12
- added joint Link0_Link6: type revolute, parent Link0, child Link6, origin xyz=0.0 0.5 1.0 rpy=0 0 0, axis 1 0 0, limit lower=-3.14159 upper=3.14159 effort=0.0 velocity=0.0
- added joint Link1_Link3: type revolute, parent Link1, child Link3, origin xyz=0 0 1 rpy=0 0 0, axis 0 0 1, limit lower=-3.14159 upper=3.14159 effort=0.0 velocity=0.0
- added joint Link1_Link4: type revolute, parent Link1, child Link4, origin xyz=-0.5 0.0 0.5 rpy=0 0 0, axis 0 1 0, limit lower=-3.14159 upper=3.14159 effort=0.0 velocity=0.0
- added joint Link1_Link8: type revolute, parent Link1, child Link8, origin xyz=0.5 0.0 0.5 rpy=0 0 0, axis 0 1 0, limit lower=-3.14159 upper=3.14159 effort=0.0 velocity=0.0
- added joint Link5_Link7: type revolute, parent Link5, child Link7, origin xyz=-0.5 -0.5 0.0 rpy=0 0 0, axis 1 0 0, limit lower=-3.14159 upper=3.14159 effort=0.0 velocity=0.0
- joint Link0_Link2: origin xyz=0.0 0.5 1.0 rpy=0 0 0 -> xyz=0.0 -0.5 1.0 rpy=0 0 0

File: body10.urdf (robot description, URDF)
Before this commit: robot robot, 11 links, 10 joints
Links:
- added link Link11, mass 1; collision box size=1 1 1; visual box size=1 1 1
Joints:
- removed joint Link0_Link7
- removed joint Link0_Link8
- removed joint Link2_Link4
- removed joint Link3_Link6
- removed joint Link4_Link5
- removed joint Link4_Link9
- removed joint Link8_Link10
- added joint Link0_Link5: type revolute, parent Link0, child Link5, origin xyz=0.0 0.0 1.5 rpy=0 0 0, axis 0 0 1, limit lower=-3.14159 upper=3.14159 effort=0.0 velocity=0.0
- added joint Link1_Link4: type revolute, parent Link1, child Link4, origin xyz=-0.5 0.5 0.0 rpy=0 0 0, axis 0 1 0, limit lower=-3.14159 upper=3.14159 effort=0.0 velocity=0.0
- added joint Link1_Link8: type revolute, parent Link1, child Link8, origin xyz=0 1 0 rpy=0 0 0, axis 1 0 0, limit lower=-3.14159 upper=3.14159 effort=0.0 velocity=0.0
- added joint Link4_Link6: type revolute, parent Link4, child Link6, origin xyz=-0.5 -0.5 0.0 rpy=0 0 0, axis 1 0 0, limit lower=-3.14159 upper=3.14159 effort=0.0 velocity=0.0
- added joint Link5_Link10: type revolute, parent Link5, child Link10, origin xyz=0.0 -0.5 0.5 rpy=0 0 0, axis 1 0 0, limit lower=-3.14159 upper=3.14159 effort=0.0 velocity=0.0
- added joint Link5_Link7: type revolute, parent Link5, child Link7, origin xyz=0.5 0.0 0.5 rpy=0 0 0, axis 0 1 0, limit lower=-3.14159 upper=3.14159 effort=0.0 velocity=0.0
- added joint Link7_Link11: type revolute, parent Link7, child Link11, origin xyz=1 0 0 rpy=0 0 0, axis 0 1 0, limit lower=-3.14159 upper=3.14159 effort=0.0 velocity=0.0
- added joint Link7_Link9: type revolute, parent Link7, child Link9, origin xyz=0.5 0.0 0.5 rpy=0 0 0, axis 0 0 1, limit lower=-3.14159 upper=3.14159 effort=0.0 velocity=0.0
- joint Link0_Link1: axis 0 0 1 -> 1 0 0; origin xyz=0.0 0.0 1.5 rpy=0 0 0 -> xyz=0.0 0.5 1.0 rpy=0 0 0
- joint Link1_Link2: axis 0 0 1 -> 0 1 0; origin xyz=0 0 1 rpy=0 0 0 -> xyz=0.5 0.5 0.0 rpy=0 0 0
- joint Link2_Link3: axis 0 1 0 -> 0 0 1

File: body11.urdf (robot description, URDF)
Before this commit: robot robot, 11 links, 10 joints
Links:
- added link Link11, mass 1; collision box size=1 1 1; visual box size=1 1 1
Joints:
- removed joint Link0_Link7
- removed joint Link1_Link2
- removed joint Link2_Link3
- removed joint Link2_Link4
- removed joint Link3_Link6
- removed joint Link4_Link5
- removed joint Link4_Link9
- removed joint Link8_Link10
- added joint Link0_Link2: type revolute, parent Link0, child Link2, origin xyz=0.0 -0.5 1.0 rpy=0 0 0, axis 1 0 0, limit lower=-3.14159 upper=3.14159 effort=0.0 velocity=0.0
- added joint Link0_Link3: type revolute, parent Link0, child Link3, origin xyz=-0.5 0.0 1.0 rpy=0 0 0, axis 0 1 0, limit lower=-3.14159 upper=3.14159 effort=0.0 velocity=0.0
- added joint Link2_Link10: type revolute, parent Link2, child Link10, origin xyz=0.5 -0.5 0.0 rpy=0 0 0, axis 0 1 0, limit lower=-3.14159 upper=3.14159 effort=0.0 velocity=0.0
- added joint Link2_Link11: type revolute, parent Link2, child Link11, origin xyz=0 -1 0 rpy=0 0 0, axis 1 0 0, limit lower=-3.14159 upper=3.14159 effort=0.0 velocity=0.0
- added joint Link3_Link4: type revolute, parent Link3, child Link4, origin xyz=-0.5 -0.5 0.0 rpy=0 0 0, axis 1 0 0, limit lower=-3.14159 upper=3.14159 effort=0.0 velocity=0.0
- added joint Link3_Link5: type revolute, parent Link3, child Link5, origin xyz=-0.5 0.0 0.5 rpy=0 0 0, axis 0 0 1, limit lower=-3.14159 upper=3.14159 effort=0.0 velocity=0.0
- added joint Link4_Link6: type revolute, parent Link4, child Link6, origin xyz=-0.5 -0.5 0.0 rpy=0 0 0, axis 0 1 0, limit lower=-3.14159 upper=3.14159 effort=0.0 velocity=0.0
- added joint Link5_Link7: type revolute, parent Link5, child Link7, origin xyz=-0.5 0.0 0.5 rpy=0 0 0, axis 0 1 0, limit lower=-3.14159 upper=3.14159 effort=0.0 velocity=0.0
- added joint Link8_Link9: type revolute, parent Link8, child Link9, origin xyz=1 0 0 rpy=0 0 0, axis 0 1 0, limit lower=-3.14159 upper=3.14159 effort=0.0 velocity=0.0
- joint Link0_Link8: axis 1 0 0 -> 0 1 0; origin xyz=0.0 -0.5 1.0 rpy=0 0 0 -> xyz=0.5 0.0 1.0 rpy=0 0 0

File: body12.urdf (robot description, URDF)
Before this commit: robot robot, 11 links, 10 joints
Joints:
- removed joint Link0_Link7
- removed joint Link0_Link8
- removed joint Link2_Link3
- removed joint Link2_Link4
- removed joint Link4_Link5
- removed joint Link4_Link9
- removed joint Link8_Link10
- added joint Link0_Link3: type revolute, parent Link0, child Link3, origin xyz=-0.5 0.0 1.0 rpy=0 0 0, axis 0 1 0, limit lower=-3.14159 upper=3.14159 effort=0.0 velocity=0.0
- added joint Link0_Link5: type revolute, parent Link0, child Link5, origin xyz=0.0 0.0 1.5 rpy=0 0 0, axis 0 0 1, limit lower=-3.14159 upper=3.14159 effort=0.0 velocity=0.0
- added joint Link1_Link4: type revolute, parent Link1, child Link4, origin xyz=-0.5 -0.5 0.0 rpy=0 0 0, axis 0 1 0, limit lower=-3.14159 upper=3.14159 effort=0.0 velocity=0.0
- added joint Link1_Link7: type revolute, parent Link1, child Link7, origin xyz=0.5 -0.5 0.0 rpy=0 0 0, axis 0 1 0, limit lower=-3.14159 upper=3.14159 effort=0.0 velocity=0.0
- added joint Link1_Link8: type revolute, parent Link1, child Link8, origin xyz=0.0 -0.5 0.5 rpy=0 0 0, axis 0 0 1, limit lower=-3.14159 upper=3.14159 effort=0.0 velocity=0.0
- added joint Link5_Link10: type revolute, parent Link5, child Link10, origin xyz=0.0 0.5 0.5 rpy=0 0 0, axis 1 0 0, limit lower=-3.14159 upper=3.14159 effort=0.0 velocity=0.0
- added joint Link7_Link9: type revolute, parent Link7, child Link9, origin xyz=0.5 0.5 0.0 rpy=0 0 0, axis 1 0 0, limit lower=-3.14159 upper=3.14159 effort=0.0 velocity=0.0
- joint Link0_Link1: axis 0 0 1 -> 1 0 0; origin xyz=0.0 0.0 1.5 rpy=0 0 0 -> xyz=0.0 -0.5 1.0 rpy=0 0 0
- joint Link1_Link2: axis 0 0 1 -> 1 0 0; origin xyz=0 0 1 rpy=0 0 0 -> xyz=0 -1 0 rpy=0 0 0
- joint Link3_Link6: axis 0 1 0 -> 1 0 0; origin xyz=1 0 0 rpy=0 0 0 -> xyz=-0.5 0.5 0.0 rpy=0 0 0

File: body13.urdf (robot description, URDF)
Before this commit: robot robot, 11 links, 10 joints
Links:
- added link Link11, mass 1; collision box size=1 1 1; visual box size=1 1 1
Joints:
- removed joint Link0_Link7
- removed joint Link0_Link8
- removed joint Link1_Link2
- removed joint Link2_Link3
- removed joint Link4_Link5
- removed joint Link4_Link9
- removed joint Link8_Link10
- added joint Link0_Link2: type revolute, parent Link0, child Link2, origin xyz=0.0 -0.5 1.0 rpy=0 0 0, axis 1 0 0, limit lower=-3.14159 upper=3.14159 effort=0.0 velocity=0.0
- added joint Link0_Link5: type revolute, parent Link0, child Link5, origin xyz=0.0 0.0 1.5 rpy=0 0 0, axis 0 0 1, limit lower=-3.14159 upper=3.14159 effort=0.0 velocity=0.0
- added joint Link1_Link3: type revolute, parent Link1, child Link3, origin xyz=-0.5 -0.5 0.0 rpy=0 0 0, axis 1 0 0, limit lower=-3.14159 upper=3.14159 effort=0.0 velocity=0.0
- added joint Link1_Link7: type revolute, parent Link1, child Link7, origin xyz=-0.5 0.5 0.0 rpy=0 0 0, axis 1 0 0, limit lower=-3.14159 upper=3.14159 effort=0.0 velocity=0.0
- added joint Link3_Link11: type revolute, parent Link3, child Link11, origin xyz=0.0 -0.5 0.5 rpy=0 0 0, axis 0 0 1, limit lower=-3.14159 upper=3.14159 effort=0.0 velocity=0.0
- added joint Link6_Link9: type revolute, parent Link6, child Link9, origin xyz=-0.5 -0.5 0.0 rpy=0 0 0, axis 1 0 0, limit lower=-3.14159 upper=3.14159 effort=0.0 velocity=0.0
- added joint Link7_Link10: type revolute, parent Link7, child Link10, origin xyz=0.5 0.5 0.0 rpy=0 0 0, axis 0 1 0, limit lower=-3.14159 upper=3.14159 effort=0.0 velocity=0.0
- added joint Link7_Link8: type revolute, parent Link7, child Link8, origin xyz=0 1 0 rpy=0 0 0, axis 1 0 0, limit lower=-3.14159 upper=3.14159 effort=0.0 velocity=0.0
- joint Link0_Link1: axis 0 0 1 -> 0 1 0; origin xyz=0.0 0.0 1.5 rpy=0 0 0 -> xyz=-0.5 0.0 1.0 rpy=0 0 0
- joint Link2_Link4: origin xyz=0 0 1 rpy=0 0 0 -> xyz=0.0 -0.5 0.5 rpy=0 0 0
- joint Link3_Link6: origin xyz=1 0 0 rpy=0 0 0 -> xyz=-0.5 -0.5 0.0 rpy=0 0 0

File: body14.urdf (robot description, URDF)
Before this commit: robot robot, 11 links, 10 joints
Links:
- removed link Link10
- removed link Link8
- removed link Link9
Joints:
- removed joint Link0_Link7
- removed joint Link0_Link8
- removed joint Link1_Link2
- removed joint Link2_Link3
- removed joint Link2_Link4
- removed joint Link4_Link5
- removed joint Link4_Link9
- removed joint Link8_Link10
- added joint Link0_Link2: type revolute, parent Link0, child Link2, origin xyz=0.5 0.0 1.0 rpy=0 0 0, axis 0 1 0, limit lower=-3.14159 upper=3.14159 effort=0.0 velocity=0.0
- added joint Link1_Link3: type revolute, parent Link1, child Link3, origin xyz=0.0 0.5 0.5 rpy=0 0 0, axis 0 0 1, limit lower=-3.14159 upper=3.14159 effort=0.0 velocity=0.0
- added joint Link1_Link4: type revolute, parent Link1, child Link4, origin xyz=-0.5 0.5 0.0 rpy=0 0 0, axis 0 1 0, limit lower=-3.14159 upper=3.14159 effort=0.0 velocity=0.0
- added joint Link1_Link5: type revolute, parent Link1, child Link5, origin xyz=0 1 0 rpy=0 0 0, axis 1 0 0, limit lower=-3.14159 upper=3.14159 effort=0.0 velocity=0.0
- added joint Link4_Link7: type revolute, parent Link4, child Link7, origin xyz=-1 0 0 rpy=0 0 0, axis 0 1 0, limit lower=-3.14159 upper=3.14159 effort=0.0 velocity=0.0
- joint Link0_Link1: axis 0 0 1 -> 1 0 0; origin xyz=0.0 0.0 1.5 rpy=0 0 0 -> xyz=0.0 0.5 1.0 rpy=0 0 0
- joint Link3_Link6: axis 0 1 0 -> 0 0 1; origin xyz=1 0 0 rpy=0 0 0 -> xyz=0 0 1 rpy=0 0 0

File: body15.urdf (robot description, URDF)
Before this commit: robot robot, 11 links, 10 joints
Links:
- removed link Link10
- removed link Link8
- removed link Link9
Joints:
- removed joint Link0_Link7
- removed joint Link0_Link8
- removed joint Link1_Link2
- removed joint Link2_Link3
- removed joint Link2_Link4
- removed joint Link3_Link6
- removed joint Link4_Link5
- removed joint Link4_Link9
- removed joint Link8_Link10
- added joint Link0_Link2: type revolute, parent Link0, child Link2, origin xyz=0.0 -0.5 1.0 rpy=0 0 0, axis 1 0 0, limit lower=-3.14159 upper=3.14159 effort=0.0 velocity=0.0
- added joint Link0_Link5: type revolute, parent Link0, child Link5, origin xyz=0.0 0.5 1.0 rpy=0 0 0, axis 1 0 0, limit lower=-3.14159 upper=3.14159 effort=0.0 velocity=0.0
- added joint Link1_Link3: type revolute, parent Link1, child Link3, origin xyz=0.5 0.0 0.5 rpy=0 0 0, axis 0 0 1, limit lower=-3.14159 upper=3.14159 effort=0.0 velocity=0.0
- added joint Link3_Link4: type revolute, parent Link3, child Link4, origin xyz=0.0 -0.5 0.5 rpy=0 0 0, axis 1 0 0, limit lower=-3.14159 upper=3.14159 effort=0.0 velocity=0.0
- added joint Link4_Link6: type revolute, parent Link4, child Link6, origin xyz=0.0 -0.5 -0.5 rpy=0 0 0, axis 0 0 1, limit lower=-3.14159 upper=3.14159 effort=0.0 velocity=0.0
- added joint Link4_Link7: type revolute, parent Link4, child Link7, origin xyz=0.0 -0.5 0.5 rpy=0 0 0, axis 0 0 1, limit lower=-3.14159 upper=3.14159 effort=0.0 velocity=0.0
- joint Link0_Link1: axis 0 0 1 -> 0 1 0; origin xyz=0.0 0.0 1.5 rpy=0 0 0 -> xyz=0.5 0.0 1.0 rpy=0 0 0

File: body16.urdf (robot description, URDF)
Before this commit: robot robot, 11 links, 10 joints
Links:
- removed link Link10
Joints:
- removed joint Link0_Link7
- removed joint Link0_Link8
- removed joint Link2_Link3
- removed joint Link2_Link4
- removed joint Link3_Link6
- removed joint Link4_Link5
- removed joint Link4_Link9
- removed joint Link8_Link10
- added joint Link0_Link4: type revolute, parent Link0, child Link4, origin xyz=0.5 0.0 1.0 rpy=0 0 0, axis 0 1 0, limit lower=-3.14159 upper=3.14159 effort=0.0 velocity=0.0
- added joint Link0_Link6: type revolute, parent Link0, child Link6, origin xyz=0.0 0.5 1.0 rpy=0 0 0, axis 1 0 0, limit lower=-3.14159 upper=3.14159 effort=0.0 velocity=0.0
- added joint Link1_Link3: type revolute, parent Link1, child Link3, origin xyz=-0.5 -0.5 0.0 rpy=0 0 0, axis 1 0 0, limit lower=-3.14159 upper=3.14159 effort=0.0 velocity=0.0
- added joint Link3_Link5: type revolute, parent Link3, child Link5, origin xyz=0.5 -0.5 0.0 rpy=0 0 0, axis 0 1 0, limit lower=-3.14159 upper=3.14159 effort=0.0 velocity=0.0
- added joint Link3_Link7: type revolute, parent Link3, child Link7, origin xyz=0 -1 0 rpy=0 0 0, axis 1 0 0, limit lower=-3.14159 upper=3.14159 effort=0.0 velocity=0.0
- added joint Link4_Link8: type revolute, parent Link4, child Link8, origin xyz=0.5 -0.5 0.0 rpy=0 0 0, axis 1 0 0, limit lower=-3.14159 upper=3.14159 effort=0.0 velocity=0.0
- added joint Link7_Link9: type revolute, parent Link7, child Link9, origin xyz=0.0 -0.5 0.5 rpy=0 0 0, axis 0 0 1, limit lower=-3.14159 upper=3.14159 effort=0.0 velocity=0.0
- joint Link0_Link1: axis 0 0 1 -> 0 1 0; origin xyz=0.0 0.0 1.5 rpy=0 0 0 -> xyz=-0.5 0.0 1.0 rpy=0 0 0
- joint Link1_Link2: axis 0 0 1 -> 1 0 0; origin xyz=0 0 1 rpy=0 0 0 -> xyz=-0.5 0.5 0.0 rpy=0 0 0

File: body17.urdf (robot description, URDF)
Before this commit: robot robot, 11 links, 10 joints
Links:
- removed link Link10
Joints:
- removed joint Link0_Link7
- removed joint Link0_Link8
- removed joint Link1_Link2
- removed joint Link2_Link3
- removed joint Link3_Link6
- removed joint Link4_Link5
- removed joint Link4_Link9
- removed joint Link8_Link10
- added joint Link0_Link2: type revolute, parent Link0, child Link2, origin xyz=0.5 0.0 1.0 rpy=0 0 0, axis 0 1 0, limit lower=-3.14159 upper=3.14159 effort=0.0 velocity=0.0
- added joint Link0_Link3: type revolute, parent Link0, child Link3, origin xyz=-0.5 0.0 1.0 rpy=0 0 0, axis 0 1 0, limit lower=-3.14159 upper=3.14159 effort=0.0 velocity=0.0
- added joint Link0_Link9: type revolute, parent Link0, child Link9, origin xyz=0.0 -0.5 1.0 rpy=0 0 0, axis 1 0 0, limit lower=-3.14159 upper=3.14159 effort=0.0 velocity=0.0
- added joint Link2_Link6: type revolute, parent Link2, child Link6, origin xyz=0.5 0.5 0.0 rpy=0 0 0, axis 1 0 0, limit lower=-3.14159 upper=3.14159 effort=0.0 velocity=0.0
- added joint Link3_Link5: type revolute, parent Link3, child Link5, origin xyz=-0.5 0.5 0.0 rpy=0 0 0, axis 1 0 0, limit lower=-3.14159 upper=3.14159 effort=0.0 velocity=0.0
- added joint Link5_Link7: type revolute, parent Link5, child Link7, origin xyz=-0.5 0.5 0.0 rpy=0 0 0, axis 0 1 0, limit lower=-3.14159 upper=3.14159 effort=0.0 velocity=0.0
- added joint Link6_Link8: type revolute, parent Link6, child Link8, origin xyz=0.0 0.5 0.5 rpy=0 0 0, axis 0 0 1, limit lower=-3.14159 upper=3.14159 effort=0.0 velocity=0.0
- joint Link2_Link4: origin xyz=0 0 1 rpy=0 0 0 -> xyz=0.5 0.0 0.5 rpy=0 0 0

File: body18.urdf (robot description, URDF)
Before this commit: robot robot, 11 links, 10 joints
Links:
- added link Link11, mass 1; collision box size=1 1 1; visual box size=1 1 1
Joints:
- removed joint Link0_Link8
- removed joint Link1_Link2
- removed joint Link2_Link3
- removed joint Link4_Link5
- removed joint Link4_Link9
- removed joint Link8_Link10
- added joint Link0_Link2: type revolute, parent Link0, child Link2, origin xyz=0.0 0.0 1.5 rpy=0 0 0, axis 0 0 1, limit lower=-3.14159 upper=3.14159 effort=0.0 velocity=0.0
- added joint Link10_Link11: type revolute, parent Link10, child Link11, origin xyz=0.5 0.5 0.0 rpy=0 0 0, axis 0 1 0, limit lower=-3.14159 upper=3.14159 effort=0.0 velocity=0.0
- added joint Link1_Link3: type revolute, parent Link1, child Link3, origin xyz=-0.5 0.5 0.0 rpy=0 0 0, axis 1 0 0, limit lower=-3.14159 upper=3.14159 effort=0.0 velocity=0.0
- added joint Link3_Link5: type revolute, parent Link3, child Link5, origin xyz=0.0 0.5 0.5 rpy=0 0 0, axis 0 0 1, limit lower=-3.14159 upper=3.14159 effort=0.0 velocity=0.0
- added joint Link5_Link10: type revolute, parent Link5, child Link10, origin xyz=0.0 0.5 0.5 rpy=0 0 0, axis 1 0 0, limit lower=-3.14159 upper=3.14159 effort=0.0 velocity=0.0
- added joint Link6_Link9: type revolute, parent Link6, child Link9, origin xyz=-0.5 0.5 0.0 rpy=0 0 0, axis 1 0 0, limit lower=-3.14159 upper=3.14159 effort=0.0 velocity=0.0
- added joint Link7_Link8: type revolute, parent Link7, child Link8, origin xyz=-0.5 -0.5 0.0 rpy=0 0 0, axis 0 1 0, limit lower=-3.14159 upper=3.14159 effort=0.0 velocity=0.0
- joint Link0_Link1: axis 0 0 1 -> 0 1 0; origin xyz=0.0 0.0 1.5 rpy=0 0 0 -> xyz=-0.5 0.0 1.0 rpy=0 0 0
- joint Link0_Link7: origin xyz=0.0 0.5 1.0 rpy=0 0 0 -> xyz=0.0 -0.5 1.0 rpy=0 0 0
- joint Link2_Link4: axis 0 0 1 -> 0 1 0; origin xyz=0 0 1 rpy=0 0 0 -> xyz=-0.5 0.0 0.5 rpy=0 0 0
- joint Link3_Link6: origin xyz=1 0 0 rpy=0 0 0 -> xyz=-0.5 0.5 0.0 rpy=0 0 0

File: body19.urdf (robot description, URDF)
Before this commit: robot robot, 11 links, 10 joints
Links:
- removed link Link10
Joints:
- removed joint Link0_Link8
- removed joint Link1_Link2
- removed joint Link2_Link4
- removed joint Link4_Link5
- removed joint Link4_Link9
- removed joint Link8_Link10
- added joint Link0_Link2: type revolute, parent Link0, child Link2, origin xyz=-0.5 0.0 1.0 rpy=0 0 0, axis 0 1 0, limit lower=-3.14159 upper=3.14159 effort=0.0 velocity=0.0
- added joint Link1_Link4: type revolute, parent Link1, child Link4, origin xyz=-0.5 -0.5 0.0 rpy=0 0 0, axis 0 1 0, limit lower=-3.14159 upper=3.14159 effort=0.0 velocity=0.0
- added joint Link3_Link5: type revolute, parent Link3, child Link5, origin xyz=-0.5 -0.5 0.0 rpy=0 0 0, axis 1 0 0, limit lower=-3.14159 upper=3.14159 effort=0.0 velocity=0.0
- added joint Link5_Link8: type revolute, parent Link5, child Link8, origin xyz=0.0 -0.5 0.5 rpy=0 0 0, axis 0 0 1, limit lower=-3.14159 upper=3.14159 effort=0.0 velocity=0.0
- added joint Link5_Link9: type revolute, parent Link5, child Link9, origin xyz=0 -1 0 rpy=0 0 0, axis 1 0 0, limit lower=-3.14159 upper=3.14159 effort=0.0 velocity=0.0
- joint Link0_Link1: axis 0 0 1 -> 1 0 0; origin xyz=0.0 0.0 1.5 rpy=0 0 0 -> xyz=0.0 -0.5 1.0 rpy=0 0 0
- joint Link2_Link3: origin xyz=0.5 0.0 0.5 rpy=0 0 0 -> xyz=-1 0 0 rpy=0 0 0
- joint Link3_Link6: axis 0 1 0 -> 1 0 0; origin xyz=1 0 0 rpy=0 0 0 -> xyz=-0.5 0.5 0.0 rpy=0 0 0

File: body2.urdf (robot description, URDF)
Before this commit: robot robot, 11 links, 10 joints
Links:
- removed link Link10
Joints:
- removed joint Link0_Link7
- removed joint Link0_Link8
- removed joint Link1_Link2
- removed joint Link2_Link4
- removed joint Link3_Link6
- removed joint Link4_Link5
- removed joint Link4_Link9
- removed joint Link8_Link10
- added joint Link0_Link2: type revolute, parent Link0, child Link2, origin xyz=0.0 -0.5 1.0 rpy=0 0 0, axis 1 0 0, limit lower=-3.14159 upper=3.14159 effort=0.0 velocity=0.0
- added joint Link1_Link4: type revolute, parent Link1, child Link4, origin xyz=0 1 0 rpy=0 0 0, axis 1 0 0, limit lower=-3.14159 upper=3.14159 effort=0.0 velocity=0.0
- added joint Link1_Link6: type revolute, parent Link1, child Link6, origin xyz=0.5 0.5 0.0 rpy=0 0 0, axis 0 1 0, limit lower=-3.14159 upper=3.14159 effort=0.0 velocity=0.0
- added joint Link2_Link7: type revolute, parent Link2, child Link7, origin xyz=0.0 -0.5 0.5 rpy=0 0 0, axis 0 0 1, limit lower=-3.14159 upper=3.14159 effort=0.0 velocity=0.0
- added joint Link3_Link5: type revolute, parent Link3, child Link5, origin xyz=0.5 0.0 0.5 rpy=0 0 0, axis 0 0 1, limit lower=-3.14159 upper=3.14159 effort=0.0 velocity=0.0
- added joint Link5_Link9: type revolute, parent Link5, child Link9, origin xyz=0.0 0.5 0.5 rpy=0 0 0, axis 1 0 0, limit lower=-3.14159 upper=3.14159 effort=0.0 velocity=0.0
- added joint Link7_Link8: type revolute, parent Link7, child Link8, origin xyz=0.0 0.5 0.5 rpy=0 0 0, axis 1 0 0, limit lower=-3.14159 upper=3.14159 effort=0.0 velocity=0.0
- joint Link0_Link1: axis 0 0 1 -> 1 0 0; origin xyz=0.0 0.0 1.5 rpy=0 0 0 -> xyz=0.0 0.5 1.0 rpy=0 0 0
- joint Link2_Link3: origin xyz=0.5 0.0 0.5 rpy=0 0 0 -> xyz=0.5 -0.5 0.0 rpy=0 0 0

File: body3.urdf (robot description, URDF)
Before this commit: robot robot, 11 links, 10 joints
Links:
- removed link Link10
- removed link Link8
- removed link Link9
Joints:
- removed joint Link0_Link7
- removed joint Link0_Link8
- removed joint Link2_Link3
- removed joint Link2_Link4
- removed joint Link3_Link6
- removed joint Link4_Link5
- removed joint Link4_Link9
- removed joint Link8_Link10
- added joint Link0_Link3: type revolute, parent Link0, child Link3, origin xyz=0.5 0.0 1.0 rpy=0 0 0, axis 0 1 0, limit lower=-3.14159 upper=3.14159 effort=0.0 velocity=0.0
- added joint Link0_Link5: type revolute, parent Link0, child Link5, origin xyz=0.0 0.0 1.5 rpy=0 0 0, axis 0 0 1, limit lower=-3.14159 upper=3.14159 effort=0.0 velocity=0.0
- added joint Link1_Link4: type revolute, parent Link1, child Link4, origin xyz=0.5 0.5 0.0 rpy=0 0 0, axis 0 1 0, limit lower=-3.14159 upper=3.14159 effort=0.0 velocity=0.0
- added joint Link2_Link6: type revolute, parent Link2, child Link6, origin xyz=-0.5 0.5 0.0 rpy=0 0 0, axis 1 0 0, limit lower=-3.14159 upper=3.14159 effort=0.0 velocity=0.0
- added joint Link2_Link7: type revolute, parent Link2, child Link7, origin xyz=-0.5 0.0 0.5 rpy=0 0 0, axis 0 0 1, limit lower=-3.14159 upper=3.14159 effort=0.0 velocity=0.0
- joint Link0_Link1: axis 0 0 1 -> 1 0 0; origin xyz=0.0 0.0 1.5 rpy=0 0 0 -> xyz=0.0 0.5 1.0 rpy=0 0 0
- joint Link1_Link2: axis 0 0 1 -> 0 1 0; origin xyz=0 0 1 rpy=0 0 0 -> xyz=-0.5 0.5 0.0 rpy=0 0 0
